File: Kilsyth.sch (KiCad schematic (older format))
At the start: 54 parts

Commit message: wip
Parts:
- removed R?: 146K, symbol Device:R_Small
- removed R?: 20K, symbol Device:R_Small
- added D?: LED, symbol Device:LED
- added J?: Conn_02x20_Counter_Clockwise, symbol Connector_Generic:Conn_02x20_Counter_Clockwise
- added R? (x3): 0R, symbol Device:R_Small
- added R?: 2K, symbol Device:R_Small
- added R? (x2): 4.7K, symbol Device:R_Small
- R10: renamed from R?; value 8.67K -> 3.3K
- R5: renamed from R?; value 20K -> 15K
- R6: renamed from R?; value 24K -> 18K
- R7: renamed from R?; value 31.6K -> 15K
- R8: renamed from R?; value 20K -> 4.7K
- R9: renamed from R?; value 39K -> 15K
- U2: renamed from U?; footprint (none) -> lfe5bg381:BGA-381_pitch0.8mm_dia0.4mm
- gave numbers to parts that had none: 33
Connections:
- wire segments 415 -> 445
- no-connect marks 5 -> 6
Other:
- note added: "RESET, PGOOD and VDIV can be left NC\nsince we don't need those features."
- note added: "Ra = Rb * (0.6 / (Vout - 0.6))\nVout = (1 + 15e3/18e3) * 0.6 = 1.1V"
- note added: "Ra = Rb * (0.6 / (Vout - 0.6))\nVout = (1 + 15e3/3.3e3) * 0.6 = 3.33V"
- note added: "Ra = Rb * (0.6 / (Vout - 0.6))\nVout = (1 + 15e3/4.7e3) * 0.6 = 2.51V"
- note removed: "Ra = Rb * (0.6 / (Vout - 0.6))\nVout = 1.1\nRa = 20K\nRb = 24K"
- note removed: "Ra = Rb * (0.6 / (Vout - 0.6))\nVout = 2.5\nRa = 31.6K\nRb = 10K"
- note removed: "Ra = Rb * (0.6 / (Vout - 0.6))\nVout = 3.3\nRa = 39K\nRb = 8.67K"
- moved on the sheet: TP1, TP2, TP3, U2G, U2J

Commit message: More progress
Parts:
- removed J?: Conn_02x20_Counter_Clockwise, symbol Connector_Generic:Conn_02x20_Counter_Clockwise
- removed U2: LFE5U-85F-6BG381C, lfe5bg381:BGA-381_pitch0.8mm_dia0.4mm, symbol lfe5bg381:LFE5U-85F-6BG381C
- added C25, C6: 22u, Capacitor_SMD:C_0603_1608Metric, symbol Device:C_Small
- added C26, C27, C28, C31: 100n, Capacitor_SMD:C_0603_1608Metric, symbol Device:C_Small
- added C29, C30: 18p, Capacitor_SMD:C_0603_1608Metric, symbol Device:C_Small
- added C32: 4u7, Capacitor_SMD:C_0603_1608Metric, symbol Device:C_Small
- added C5: 10u, Capacitor_SMD:C_0603_1608Metric, symbol Device:C_Small
- added FB1: Ferrite_Bead_Small, Inductor_SMD:L_0603_1608Metric, symbol Device:Ferrite_Bead_Small
- added J1: Conn_02x20_Odd_Even, symbol Connector_Generic:Conn_02x20_Odd_Even
- added J2: USB_B_Micro, Connector_USB:USB_Micro-B_Molex_47346-0001, symbol Connector:USB_B_Micro
- added J3: USB_C_Receptacle, JAE-USB-C:USBC_DX07S024JJ2R1300, symbol Connector:USB_C_Receptacle
- added J4: Conn_JTAG, Connector_PinSocket_2.54mm:PinSocket_2x03_P2.54mm_Vertical_SMD, symbol Connector_Generic:Conn_02x03_Counter_Clockwise
- added J5: PUSB3FR4Z, PUSB3FR4Z:PUSB3FR4Z, symbol Connector_Generic:Conn_02x05_Counter_Clockwise
- added R16: 0R, Resistor_SMD:R_0603_1608Metric, symbol Device:R_Small
- added R18, R19: 5K1, Resistor_SMD:R_0603_1608Metric, symbol Device:R
- added R20, R21, R22, R23, R28, R29, R30, R31, R32, R33, R34, R35, R36, R37, R38, R39, R40, R41, R42, R43, R44, R45, R46, R47, R48, R49, R50, R51: 0R, Resistor_SMD:R_0603_1608Metric, symbol Device:R
- added R24: 1.6K, Resistor_SMD:R_0603_1608Metric, symbol Device:R_Small
- added R25, R26, R27: 10K, Resistor_SMD:R_0603_1608Metric, symbol Device:R
- added R52, R53: 1M, Resistor_SMD:R_0603_1608Metric, symbol Device:R_Small
- added R54: 4k7, Resistor_SMD:R_0603_1608Metric, symbol Device:R_Small
- added TP3: TestPoint, TestPoint:TestPoint_Pad_D1.0mm, symbol Connector:TestPoint
- added U2: MIC5504-1.8YM5, Package_TO_SOT_SMD:SOT-23-5, symbol Regulator_Linear:MIC5504-1.8YM5
- added U3: LFE5U-85F-6BG381C, lfe5bg381:BGA-381_pitch0.8mm_dia0.4mm, symbol lfe5bg381:LFE5U-85F-6BG381C
- added U4: FT600Q, Package_DFN_QFN:QFN-56-1EP_7x7mm_P0.4mm_EP5.7x5.7mm, symbol FT600Q:FT600Q
- added U5: IS25LP128F-JBLE, SOA008-150mil:SOA008-150-208mil, symbol Memory_EEPROM:25LCxxx
- added Y1: 30MHz ±20ppm, Crystal:Crystal_SMD_2016-4Pin_2.0x1.6mm, symbol Device:Crystal_GND24_Small
- C1, C2, C3, C4: footprint (none) -> Capacitor_SMD:C_0603_1608Metric
- C10: renamed from C8; footprint (none) -> Capacitor_SMD:C_0603_1608Metric
- C11: renamed from C9; footprint (none) -> Capacitor_SMD:C_0603_1608Metric
- C12: renamed from C10; footprint (none) -> Capacitor_SMD:C_0603_1608Metric
- C13: renamed from C11; footprint (none) -> Capacitor_SMD:C_0603_1608Metric
- C14: renamed from C12; footprint (none) -> Capacitor_SMD:C_0603_1608Metric
- C15: renamed from C13; footprint (none) -> Capacitor_SMD:C_0603_1608Metric
- C16: renamed from C14; footprint (none) -> Capacitor_SMD:C_0603_1608Metric
- C17: renamed from C15; footprint (none) -> Capacitor_SMD:C_0603_1608Metric
- C18: renamed from C16; footprint (none) -> Capacitor_SMD:C_0603_1608Metric
- C19: renamed from C17; footprint (none) -> Capacitor_SMD:C_0603_1608Metric
- C20: renamed from C18; footprint (none) -> Capacitor_SMD:C_0603_1608Metric
- C21: renamed from C19; footprint (none) -> Capacitor_SMD:C_0603_1608Metric
- C22: renamed from C20; footprint (none) -> Capacitor_SMD:C_0603_1608Metric
- C23: renamed from C21; footprint (none) -> Capacitor_SMD:C_0603_1608Metric
- C24: renamed from C22; footprint (none) -> Capacitor_SMD:C_0603_1608Metric
- C7: renamed from C5; footprint (none) -> Capacitor_SMD:C_0603_1608Metric
- C8: renamed from C6; footprint (none) -> Capacitor_SMD:C_0603_1608Metric
- C9: renamed from C7; footprint (none) -> Capacitor_SMD:C_0603_1608Metric
- D1: renamed from D?; footprint (none) -> LED_SMD:LED_0603_1608Metric
- L1, L2, L3: footprint (none) -> Inductor_SMD:L_0603_1608Metric
- R1: footprint (none) -> Resistor_SMD:R_0603_1608Metric
- R10: renamed from R7; footprint (none) -> Resistor_SMD:R_0603_1608Metric
- R11: renamed from R8; footprint (none) -> Resistor_SMD:R_0603_1608Metric
- R12: renamed from R9; footprint (none) -> Resistor_SMD:R_0603_1608Metric
- R13: renamed from R10; footprint (none) -> Resistor_SMD:R_0603_1608Metric
- R14, R15, R17, R2, R3, R4: renamed from R?; footprint (none) -> Resistor_SMD:R_0603_1608Metric
- R5: renamed from R2; footprint (none) -> Resistor_SMD:R_0603_1608Metric
- R6: renamed from R3; footprint (none) -> Resistor_SMD:R_0603_1608Metric
- R7: renamed from R4; footprint (none) -> Resistor_SMD:R_0603_1608Metric
- R8: renamed from R5; footprint (none) -> Resistor_SMD:R_0603_1608Metric
- R9: renamed from R6; footprint (none) -> Resistor_SMD:R_0603_1608Metric
- TP1: renamed from TP2; footprint (none) -> TestPoint:TestPoint_Pad_D1.0mm
- TP2: renamed from TP3; footprint (none) -> TestPoint:TestPoint_Pad_D1.0mm
- TP4: renamed from TP1; footprint (none) -> TestPoint:TestPoint_Pad_D1.0mm
- U1: footprint (none) -> Package_QFP:LQFP-32_5x5mm_P0.5mm
Connections:
- net labels added: +1V8, FT_BE_0, FT_BE_1, FT_CLK, FT_DATA_0, FT_DATA_1, FT_DATA_10, FT_DATA_11, FT_DATA_12, FT_DATA_13, FT_DATA_14, FT_DATA_15, FT_DATA_2, FT_DATA_3, FT_DATA_4, FT_DATA_5, FT_DATA_6, FT_DATA_7, FT_DATA_8, FT_DATA_9, FT_DM, FT_DP, FT_GPIO0, FT_GPIO1, FT_OE_N, FT_RD_N, FT_RIDN, FT_RIDP, FT_RXF_N, FT_TODN, FT_TODP, FT_TXE_N, FT_WR_N, JTAG_TCK, JTAG_TDI, JTAG_TDO, JTAG_TMS, USB_DM, USB_DP, USB_VBUS, VBUS
- wire segments 445 -> 669
- no-connect marks 6 -> 21
Other:
- note added: "1.1V rail. Max 3A"
- note added: "1.8V rail. Max 300mA"
- note added: "2.5V rail. Max 2A"
- note added: "3.3V rail. Max 2A"
- note added: "No idea if these are needed\nso let's have 0R so we can patch it later."
- note added: "RESET, PGOOD and VDIV can be left NC\nsince we don't need those features.\nENx is open drain. NC = enabled."
- note removed: "RESET, PGOOD and VDIV can be left NC\nsince we don't need those features."
- moved on the sheet: D1, R17, R2, R3, R4, TP4

Commit message: more wip
Parts:
- removed C32: 4u7, Capacitor_SMD:C_0603_1608Metric, symbol Device:C_Small
- added C? (x4): 100n, Capacitor_SMD:C_0603_1608Metric, symbol Device:C_Small
- added C?: 4u7, Capacitor_SMD:C_0603_1608Metric, symbol Device:C_Small
- FB1: value Ferrite_Bead_Small -> Ferrite_Bead
- U5: Description (none) -> 128Mbit NOR memory
Connections:
- net labels added: FLASH_CSn, FLASH_HOLDn, FLASH_MISO, FLASH_MOSI, FLASH_SCK, FLASH_WPn
- wire segments 669 -> 691
Other:
- note added: "Design goals:\n\n- High speed transfers with the FT600. Should reach 190MB/s theoretically with 16 bit @ 100MHz.\n\n- Should work with any variant of LFE5U, i.e. 12F, 25F, 45F, 85F.\n\n- Low cost BOM. Ideally <$25 for everything.\n\n- Loads bitstream from flash\n\n- JTAG should work\n\n- Bootloader on flash that allows programming the rest of the flash over the FT600. Is 128Mbit enough?\n This sh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"
- note added: "FPGA Power"
- note added: "JTAG and Flash"
- note added: "USB and FT600"
- note added: "Voltage regulators"
- moved on the sheet: C26, C27, C28, C29, C30, C31, D1, FB1, J1, J2, J3, J4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

Commit message: WIP
Parts:
- removed R2: 2K, Resistor_SMD:R_0603_1608Metric, symbol Device:R_Small
- added C32: 100n, Capacitor_SMD:C_0603_1608Metric, symbol Device:C_Small
- added D?: LED, LED_SMD:LED_0603_1608Metric, symbol Device:LED
- added R? (x2): 10K, Resistor_SMD:R_0603_1608Metric, symbol Device:R_Small
- added R?: 0R, Resistor_SMD:R_0603_1608Metric, symbol Device:R
- added R? (x2): 2K, Resistor_SMD:R_0603_1608Metric, symbol Device:R_Small
- added SW?: SW_Push, symbol Switch:SW_Push
- added TP?: TestPoint, TestPoint:TestPoint_Pad_D1.0mm, symbol Connector:TestPoint
- added U6: DSC6001CI2A-016.0000T, Crystal:Crystal_SMD_3225-4Pin_3.2x2.5mm, symbol dsc6001ci2a-016.0000t:DSC6001CI2A-016.0000T
- J3: value USB_C_Receptacle -> DX07S024JJ2; Aliexpress-maybe (none) -> https://www.aliexpress.com/item/100pcs-USB-3-1-Type-C-Conne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; Datasheet2 (none) -> https://www.mouser.se/datasheet/2/206/B-0297-4E_0301-2E_DX0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; Mouser (none) -> 656-DX07S024JJ2R1300
- J5: Mouser https://www.mouser.se/ProductDetail/Nexperia/PUSB3FR4Z?qs=%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 -> 771-PUSB3FR4Z; Mouser2 (none) -> https://www.mouser.se/ProductDetail/Nexperia/PUSB3FR4Z?qs=%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
- U1: Mouser (none) -> https://www.mouser.se/ProductDetail/Texas-Instruments/TPS65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
- U1: Mouser (none) -> 595-TPS65261RHBR
- U4: Mouser (none) -> 895-FT600Q-B-T
- U5: Mouser https://www.mouser.se/ProductDetail/ISSI/IS25LP128F-JBLE?qs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 -> 870-IS25LP128F-JBLE; Mouser2 (none) -> https://www.mouser.se/ProductDetail/ISSI/IS25LP128F-JBLE?qs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
- gave numbers to parts that had none: 5
Connections:
- net labels added: CLK_16MHz, DONE, INITn, PROGRAMn
- wire segments 691 -> 741
- no-connect marks 21 -> 26
Other:
- note added: "LEDs"
- note added: "System clock"
- moved on the sheet: C33, D1, J4, R10, R12, R3, R4, R54, R8, U3B, U3G, U3J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

Commit message: WIP
Other:
- note added: "Optional"
- note added: "TODO: 10n + 100n"
Changed lines of the file:
@@
 Wire Bus Line
 	18050 6500 18050 9100
+Text Notes 8800 4600 0    50   ~ 0
+Optional
+Text Notes 2950 17950 0    50   ~ 0
+Optional
+Text Notes 18800 1950 0    50   ~ 0
+TODO: 10n + 100n
 $EndSCHEMATC

Commit message: Hmmmm
Parts:
- removed J1: Conn_02x20_Odd_Even, symbol Connector_Generic:Conn_02x20_Odd_Even
- added C32, C43: 4u7, Capacitor_SMD:C_0603_1608Metric, symbol Device:C_Small
- added C35, C36, C41, C42, C44, C45, C46, C50, C51, C54, C55, C58, C60, C62, C64, C66: 100n, Capacitor_SMD:C_0603_1608Metric, symbol Device:C_Small
- added C47, C48, C49, C52, C53, C56, C57, C59, C61, C63, C65, C67: 10n, Capacitor_SMD:C_0603_1608Metric, symbol Device:C_Small
- added H1, H2, H3, H4: (no value), MountingHole:MountingHole_3.2mm_M3_Pad, symbol Mechanical:MountingHole_Pad
- added J4: Conn_02x20_Counter_Clockwise, Connector_PinHeader_2.54mm:PinHeader_2x20_P2.54mm_Vertical_SMD, symbol Connector_Generic:Conn_02x20_Counter_Clockwise
- added J5, J8, J9: Conn_02x06_Counter_Clockwise, Connector_PinSocket_2.54mm:PinSocket_2x06_P2.54mm_Horizontal, symbol Connector_Generic:Conn_02x06_Counter_Clockwise
- added J6: PUSB3FR4Z, PUSB3FR4Z:PUSB3FR4Z, symbol Connector_Generic:Conn_02x05_Counter_Clockwise
- added U7: AS4C32M16SB, Package_SO:TSOP-II-54_22.2x10.16mm_P0.8mm, symbol AS4C32M16SB:AS4C32M16SB
- SW1: renamed from SW?; footprint (none) -> kilsyth_extra:SmallButton
- U3: renamed from U1; footprint Package_QFP:LQFP-32_5x5mm_P0.5mm -> kilsyth_extra:S-PVQFN-N32
- U6: renamed from U4; footprint Package_DFN_QFN:QFN-56-1EP_7x7mm_P0.4mm_EP5.7x5.7mm -> kilsyth_extra:QFN-56-1EP_7x7mm_P0.4mm_EP5.7x5.7mm_FIXED
- gave numbers to parts that had none: 7
- renumbered C32 to C1, C9 to C10, C10 to C11, C11 to C12, C12 to C13, C13 to C14, C14 to C15, C15 to C16, C16 to C17, C17 to C18, C18 to C19, C1 to C2, C19 to C20, C20 to C21, C21 to C22, C22 to C23, C23 to C24, C24 to C25, C25 to C26, C33 to C27, C31 to C29, C2 to C3, C26 to C30, C27 to C31, C29 to C33, C30 to C34, C34 to C37, C35 to C38, C36 to C39, C3 to C4, C37 to C40, C4 to C5, C5 to C6, C6 to C7, C7 to C8, C8 to C9, D1 to D2, J4 to J1, J3 to J2, J2 to J3, J5 to J7, R3 to R1, R9 to R10, R10 to R11, R11 to R12, R12 to R13, R13 to R14, R14 to R17, R15 to R18, R16 to R19, R1 to R2, R17 to R21, R52 to R23, R53 to R24, R18 to R25, R19 to R26, R20 to R27, R21 to R28, R22 to R29, R4 to R3, R23 to R30, R24 to R31, R25 to R32, R26 to R33, R27 to R34, R28 to R35, R29 to R36, R30 to R37, R31 to R38, R32 to R39, R54 to R4, R33 to R40, R34 to R41, R35 to R42, R36 to R43, R37 to R44, R38 to R45, R39 to R46, R40 to R47, R41 to R48, R42 to R49, R43 to R50, R44 to R51, R45 to R52, R46 to R53, R47 to R54, R48 to R55, R49 to R56, R50 to R57, R51 to R58, R8 to R9, TP1 to TP2, TP2 to TP3, TP3 to TP4, TP4 to TP5, U6 to U1, U3 to U2, U2 to U4
Connections:
- net labels added: BANK2, BANK3, BANK6, PMOD0_0, PMOD0_1, PMOD0_2, PMOD0_3, PMOD0_4, PMOD0_5, PMOD0_6, PMOD0_7, PMOD0_VCC, PMOD1_0, PMOD1_1, PMOD1_2, PMOD1_3, PMOD1_4, PMOD1_5, PMOD1_6, PMOD1_7, PMOD1_VCC, PMOD2_0, PMOD2_1, PMOD2_2, PMOD2_3, PMOD2_4, PMOD2_5, PMOD2_6, PMOD2_7, RAM_A0, RAM_A1, RAM_A10, RAM_A11, RAM_A12, RAM_A2, RAM_A3, RAM_A4, RAM_A5, RAM_A6, RAM_A7, RAM_A8, RAM_A9, RAM_BA0, RAM_BA1, RAM_CKE, RAM_CLK, RAM_DQ0, RAM_DQ1, RAM_DQ10, RAM_DQ11, RAM_DQ12, RAM_DQ13, RAM_DQ14, RAM_DQ15, RAM_DQ2, RAM_DQ3, RAM_DQ4, RAM_DQ5, RAM_DQ6, RAM_DQ7, RAM_DQ8, RAM_DQ9, RAM_DQM0, RAM_DQM1, RAM_~CAS, RAM_~CS, RAM_~RAS, RAM_~WE, USB_RXN, USB_RXP, USB_TXN, USB_TXP
- net labels removed: VBUS
- wire segments 741 -> 1152
- no-connect marks 26 -> 39
Other:
- note added: "(KiCad bug, should use VBus but can't)"
- note added: "FT600"
- note added: "One pair per bank"
- note added: "ROSC sets the switching frequency.\n73.2K = 600kHz. Lower R -> higher f"
- note added: "SDRAM"
- note removed: "TODO: 10n + 100n"
- moved on the sheet: J7, R25, R26, U2B, U2C, U2D, U2E, U2F, U2H, U2I

Commit message: Routing
Parts:
- removed C28, C29: 100n, Capacitor_SMD:C_0603_1608Metric, symbol Device:C_Small
- removed R23, R24: 1M, Resistor_SMD:R_0603_1608Metric, symbol Device:R_Small
- removed R26: 5K1, Resistor_SMD:R_0603_1608Metric, symbol Device:R
- removed R30: 0R, Resistor_SMD:R_0603_1608Metric, symbol Device:R
Connections:
- net FT_DM: now also J6.2 (Pin_2), J6.9 (Pin_9); no longer J6.4 (Pin_4), J6.7 (Pin_7)
- net FT_DP: now also J6.1 (Pin_1), J6.10 (Pin_10); no longer J6.5 (Pin_5), J6.6 (Pin_6)
- net FT_RIDN: no longer J2.A10 (RX2-)
- net FT_RIDP: no longer J2.A11 (RX2+)
- net GND: now also J2.S1 (SHIELD), J3.6 (Shield)
- net USB_DM: no longer J2.B7 (D-)
- net USB_DP: no longer J2.B6 (D+)
- net USB_TXN: no longer J2.B3 (TX2-)
- net USB_TXP: no longer J2.B2 (TX2+)
- no-connect marks 39 -> 46
Other:
- note added: "NON-reversible implementation.\nSorry for that but it's too expensive."
- moved on the sheet: R27, R28, R31

Commit message: yarrr. fixed imoprtant pmic bug
Parts:
- J3: footprint Connector_USB:USB_Micro-B_Molex_47346-0001 -> Connector_USB:USB_Micro-B_Molex-105017-0001
- L1, L2, L3: footprint Inductor_SMD:L_0603_1608Metric -> L_1008_1210:L_1008_1210
Changed lines of the file:
@@
 F 0 "L1" V 4785 3450 50  0000 C CNN
 F 1 "2.2u" V 4694 3450 50  0000 C CNN
-F 2 "Inductor_SMD:L_0603_1608Metric" H 4600 3450 50  0001 C CNN
+F 2 "L_1008_1210:L_1008_1210" H 4600 3450 50  0001 C CNN
 F 3 "~" H 4600 3450 50  0001 C CNN
 F 4 "81-DFE322512F-2R2MP2" V 4600 3450 50  0001 C CNN "Mouser"
@@
 F 0 "L2" V 4785 5250 50  0000 C CNN
 F 1 "2.2u" V 4694 5250 50  0000 C CNN
-F 2 "Inductor_SMD:L_0603_1608Metric" H 4600 5250 50  0001 C CNN
+F 2 "L_1008_1210:L_1008_1210" H 4600 5250 50  0001 C CNN
 F 3 "~" H 4600 5250 50  0001 C CNN
 F 4 "81-DFE322512F-2R2MP2" V 4600 5250 50  0001 C CNN "Mouser"
@@
 F 0 "L3" V 4785 7050 50  0000 C CNN
 F 1 "2.2u" V 4694 7050 50  0000 C CNN
-F 2 "Inductor_SMD:L_0603_1608Metric" H 4600 7050 50  0001 C CNN
+F 2 "L_1008_1210:L_1008_1210" H 4600 7050 50  0001 C CNN
 F 3 "~" H 4600 7050 50  0001 C CNN
 F 4 "81-DFE322512F-2R2MP2" V 4600 7050 50  0001 C CNN "Mouser"
@@
 F 0 "J3" H 9405 5067 50  0000 C CNN
 F 1 "USB_B_Micro" H 9405 4976 50  0000 C CNN
-F 2 "Connector_USB:USB_Micro-B_Molex_47346-0001" H 9500 4550 50  0001 C CNN
+F 2 "Connector_USB:USB_Micro-B_Molex-105017-0001" H 9500 4550 50  0001 C CNN
 F 3 "~" H 9500 4550 50  0001 C CNN
 	1    9350 4600
@@
 Wire Wire Line
 	11250 7100 11750 7100
+Connection ~ 11250 7100
+Connection ~ 11750 7100
 Wire Bus Line
 	18150 9200 21550 9200
@@
 Wire Bus Line
 	18050 6500 18050 9100
-Connection ~ 11250 7100
-Connection ~ 11750 7100
 $EndSCHEMATC
