File: Kilsyth.sch (KiCad schematic (older format))
At the start: 152 parts, among them J1 Conn_JTAG, J2 DX07S024JJ2, J3 USB_B_Micro, J4 Conn_02x20_Counter_Clockwise, J5 Conn_02x06_Counter_Clockwise, J6 PUSB3FR4Z, J7 PUSB3FR4Z, J8 Conn_02x06_Counter_Clockwise, J9 Conn_02x06_Counter_Clockwise, SW1 SW_Push, U1 DSC6001CI2A-016.0000T, U2 LFE5U-85F-6BG381C, U3 TPS65261, U4 MIC5504-1.8YM5, U5 IS25LP128F-JBLE, U6 FT600Q, U7 AS4C32M16SB, Y1 30MHz ±20ppm

Commit message: woop
Connections:
- net labels added: BANK7
- net labels removed: BANK2, BANK3
- wire segments 1117 -> 1092
- no-connect marks 46 -> 57
Other:
- moved on the sheet: C32, C35, C36, C41, C42, C43, U2C, U2D, U2E, U2F, U7

Commit message: before r0 hell
Parts:
- removed R15: 0R, Resistor_SMD:R_0603_1608Metric, symbol Device:R
- added R23, R24: 0R, Resistor_SMD:R_0603_1608Metric, symbol Device:R
Connections:
- net labels added: BANK0
- net labels removed: BANK6
- wire segments 1092 -> 1091
Other:
- moved on the sheet: U2A, U2E
Changed lines of the file:
@@
 	1    0    0    -1
 $EndComp
-Text GLabel 15050 7500 0    50   Input ~ 0
+Text GLabel 14750 7500 0    50   Input ~ 0
 FT_GPIO0
-Text GLabel 15050 7600 0    50   Input ~ 0
+Text GLabel 14750 7600 0    50   Input ~ 0
 FT_GPIO1
 Wire Wire Line
@@
 L lfe5bg381:LFE5U-85F-6BG381C U2
 U 1 1 66BE2CC2
-P 20350 7100
-F 0 "U2" H 20350 8087 60  0000 C CNN
-F 1 "LFE5U-85F-6BG381C" H 20350 7981 60  0000 C CNN
-F 2 "lfe5bg381:BGA-381_pitch0.8mm_dia0.4mm" H 19300 8050 60  0001 C CNN
-F 3 "" H 19300 8050 60  0000 C CNN
-	1    20350 7100
+P 16800 17150
+F 0 "U2" H 16800 18137 60  0000 C CNN
+F 1 "LFE5U-85F-6BG381C" H 16800 18031 60  0000 C CNN
+F 2 "lfe5bg381:BGA-381_pitch0.8mm_dia0.4mm" H 15750 18100 60  0001 C CNN
+F 3 "" H 15750 18100 60  0000 C CNN
+	1    16800 17150
 	1    0    0    -1
 $EndComp
-NoConn ~ 21100 7600
-NoConn ~ 19600 7600
-NoConn ~ 19600 7700
+NoConn ~ 28950 10500
+NoConn ~ 27450 10500
+NoConn ~ 27450 10600
 $Comp
 L lfe5bg381:LFE5U-85F-6BG381C U2
@@
 L lfe5bg381:LFE5U-85F-6BG381C U2
 U 5 1 673D53F2
-P 16800 17150
-F 0 "U2" H 16800 18137 60  0000 C CNN
-F 1 "LFE5U-85F-6BG381C" H 16800 18031 60  0000 C CNN
-F 2 "lfe5bg381:BGA-381_pitch0.8mm_dia0.4mm" H 15750 18100 60  0001 C CNN
-F 3 "" H 15750 18100 60  0000 C CNN
-	5    16800 17150
+P 20350 7100
+F 0 "U2" H 20350 8087 60  0000 C CNN
+F 1 "LFE5U-85F-6BG381C" H 20350 7981 60  0000 C CNN
+F 2 "lfe5bg381:BGA-381_pitch0.8mm_dia0.4mm" H 19300 8050 60  0001 C CNN
+F 3 "" H 19300 8050 60  0000 C CNN
+	5    20350 7100
 	1    0    0    -1
 $EndComp
-NoConn ~ 16050 18050
+NoConn ~ 19600 8000
 $Comp
 L lfe5bg381:LFE5U-85F-6BG381C U2
@@
 	6000 14100 6000 14200
 $Comp
-L Device:R R15
-U 1 1 6B048BF0
-P 5150 14650
-F 0 "R15" V 5110 14800 50  0000 L CNN
-F 1 "0R" V 5150 14650 50  0000 C CNN
-F 2 "Resistor_SMD:R_0603_1608Metric" V 5080 14650 50  0001 C CNN
-F 3 "~" H 5150 14650 50  0001 C CNN
-	1    5150 14650
-	0    1    1    0
-$EndComp
-Wire Wire Line
-	4900 14650 5000 14650
-Wire Wire Line
-	5300 14650 5650 14650
-$Comp
 L Switch:SW_Push SW1
 U 1 1 6B347A71
@@
 	18800 17900 18800 18000
 Text Label 15850 16450 2    50   ~ 0
-BANK6
+BANK0
 Text Label 18800 16500 2    50   ~ 0
 BANK7
@@
 	10150 14200 10250 14300
 NoConn ~ 21050 12750
+$Comp
+L Device:R R23
+U 1 1 60E42639
+P 14900 7500
+F 0 "R23" V 14860 7650 50  0000 L CNN
+F 1 "0R" V 14900 7500 50  0000 C CNN
+F 2 "Resistor_SMD:R_0603_1608Metric" V 14830 7500 50  0001 C CNN
+F 3 "~" H 14900 7500 50  0001 C CNN
+	1    14900 7500
+	0    1    1    0
+$EndComp
+$Comp
+L Device:R R24
+U 1 1 60E4263F
+P 14900 7600
+F 0 "R24" V 14860 7750 50  0000 L CNN
+F 1 "0R" V 14900 7600 50  0000 C CNN
+F 2 "Resistor_SMD:R_0603_1608Metric" V 14830 7600 50  0001 C CNN
+F 3 "~" H 14900 7600 50  0001 C CNN
+	1    14900 7600
+	0    1    1    0
+$EndComp
+Wire Wire Line
+	4900 14650 5650 14650
 Wire Bus Line
 	18150 9200 21550 9200
@@
 	12700 7100 12700 9100
 Wire Bus Line
-	12950 12350 12950 14200
+	18850 12750 18850 14200
 Wire Bus Line
 	21650 12550 21650 14200
 Wire Bus Line
-	18850 12750 18850 14200
+	12950 12350 12950 14200
 Wire Bus Line
 	19050 6500 19050 9100
@@
 	21650 6500 21650 9100
 Wire Bus Line
-	14350 11350 14350 14200
+	10150 12350 10150 14200
 Wire Bus Line
 	17650 11350 17650 14200
 Wire Bus Line
-	10150 12350 10150 14200
+	14350 11350 14350 14200
 Wire Bus Line
 	18050 6500 18050 9100

Commit message: ayy
Parts:
- removed J5, J8, J9: Conn_02x06_Counter_Clockwise, Connector_PinSocket_2.54mm:PinSocket_2x06_P2.54mm_Horizontal, symbol Connector_Generic:Conn_02x06_Counter_Clockwise
- added J5, J8, J9: Conn_02x06_Odd_Even, Connector_PinSocket_2.54mm:PinSocket_2x06_P2.54mm_Horizontal, symbol Connector_Generic:Conn_02x06_Odd_Even
Connections:
- net labels added: PMOD0_8, PMOD1_8, PMOD2_8, PMOD2_VCC
- net labels removed: PMOD0_0, PMOD1_0, PMOD2_0
- wire segments 1091 -> 1099
Other:
- moved on the sheet: R23, R24, R35, R36, R37, R39, R40, R41, R42, R43, R44, R45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

Commit message: puh
Parts:
- J1: footprint Connector_PinSocket_2.54mm:PinSocket_2x03_P2.54mm_Vertical_SMD -> Connector_PinHeader_2.54mm:PinHeader_2x03_P2.54mm_Vertical_SMD
Changed lines of the file:
@@
 F 0 "J1" H 2600 11717 50  0000 C CNN
 F 1 "Conn_JTAG" H 2600 11626 50  0000 C CNN
-F 2 "Connector_PinSocket_2.54mm:PinSocket_2x03_P2.54mm_Vertical_SMD" H 2550 11400 50  0001 C CNN
+F 2 "Connector_PinHeader_2.54mm:PinHeader_2x03_P2.54mm_Vertical_SMD" H 2550 11400 50  0001 C CNN
 F 3 "~" H 2550 11400 50  0001 C CNN
 	1    2550 11400

Commit message: oy
Connections:
- net RAM_DQ0: now also U2.U19 (PR89C); no longer U2.U18 (PR92A)
- net RAM_DQ14: now also U2.J17 (PR20C); no longer U2.J18 (GR_PCLK2_0)
- net RAM_DQ15: now also U2.J18 (GR_PCLK2_0); no longer U2.J17 (PR20C)
- net RAM_DQ2: now also U2.U18 (PR92A); no longer U2.U16 (GPLL0T_IN)
- net RAM_DQ3: now also U2.U16 (GPLL0T_IN); no longer U2.N18 (PR53C)
- net RAM_DQM0: now also U2.T19 (PR89A); no longer U2.U19 (PR89C)
- net RAM_~CAS: now also U2.R20 (PR86B); no longer U2.T19 (PR89A)
- net RAM_~RAS: now also U2.P18 (PR83D); no longer U2.R20 (PR86B)
Changed lines of the file:
@@
 Wire Wire Line
 	10850 13750 10250 13750
-Text Label 19550 12550 2    50   ~ 0
+Text Label 19550 12650 2    50   ~ 0
 RAM_DQ0
 Text Label 21050 12550 0    50   ~ 0
 RAM_DQ1
+Text Label 19550 12550 2    50   ~ 0
+RAM_DQ2
 Text Label 19550 12450 2    50   ~ 0
-RAM_DQ2
-Text Label 19550 13450 2    50   ~ 0
 RAM_DQ3
 Text Label 21050 13250 0    50   ~ 0
@@
 Text Label 12350 13450 0    50   ~ 0
 RAM_DQ13
+Text Label 10850 13050 2    50   ~ 0
+RAM_DQ14
 Text Label 10850 12450 2    50   ~ 0
-RAM_DQ14
-Text Label 10850 13050 2    50   ~ 0
 RAM_DQ15
-Text Label 19550 12650 2    50   ~ 0
+Text Label 19550 12750 2    50   ~ 0
 RAM_DQM0
 Text Label 10850 12750 2    50   ~ 0
@@
 Text Label 19550 12850 2    50   ~ 0
 RAM_~WE
-Text Label 19550 12750 2    50   ~ 0
+Text Label 21050 12950 0    50   ~ 0
 RAM_~CAS
-Text Label 21050 12950 0    50   ~ 0
+Text Label 21050 13050 0    50   ~ 0
 RAM_~RAS
 Text Label 19550 12950 2    50   ~ 0
@@
 	21550 7900 21650 8000
 $Comp
-L power:+3V3 #PWR?
+L power:+3V3 #PWR0117
 U 1 1 66D5A216
 P 12200 1150
-F 0 "#PWR?" H 12200 1000 50  0001 C CNN
+F 0 "#PWR0117" H 12200 1000 50  0001 C CNN
 F 1 "+3V3" H 12215 1323 50  0000 C CNN
 F 2 "" H 12200 1150 50  0001 C CNN
@@
 Wire Wire Line
 	12200 1150 12200 1350
+Connection ~ 12200 1350
 Wire Bus Line
 	18150 9200 21550 9200
@@
 Wire Bus Line
 	18050 6500 18050 9100
-Connection ~ 12200 1350
 $EndSCHEMATC

Commit message: getting somewhere
Parts:
- removed C6: 10u, Capacitor_SMD:C_0603_1608Metric, symbol Device:C_Small
- removed C7: 22u, Capacitor_SMD:C_0603_1608Metric, symbol Device:C_Small
- removed J4: Conn_02x20_Counter_Clockwise, Connector_PinHeader_2.54mm:PinHeader_2x20_P2.54mm_Vertical_SMD, symbol Connector_Generic:Conn_02x20_Counter_Clockwise
- removed R19: 0R, Resistor_SMD:R_0603_1608Metric, symbol Device:R_Small
- removed TP4: TestPoint, TestPoint:TestPoint_Pad_D1.0mm, symbol Connector:TestPoint
- removed U4: MIC5504-1.8YM5, Package_TO_SOT_SMD:SOT-23-5, symbol Regulator_Linear:MIC5504-1.8YM5
- added D10, D3, D4, D5, D6, D7, D8, D9: LED, LED_SMD:LED_0603_1608Metric, symbol Device:LED
- added J10: Conn_02x01, Connector_PinHeader_2.54mm:PinHeader_2x01_P2.54mm_Vertical, symbol Connector_Generic:Conn_02x01
- added J4: Conn_02x20_Odd_Even, Connector_PinHeader_2.54mm:PinHeader_2x20_P2.54mm_Vertical_SMD, symbol Connector_Generic:Conn_02x20_Odd_Even
- added R15, R26, R30, R59, R60, R61, R62, R63: 2K, Resistor_SMD:R_0603_1608Metric, symbol Device:R_Small
Connections:
- net +3V3: now also J5.1 (Pin_1), J5.2 (Pin_2), J8.1 (Pin_1), J8.2 (Pin_2), J9.1 (Pin_1), J9.2 (Pin_2), J10.1 (Pin_1)
- net CLK_16MHz: now also U2.G3 (PCLKT7_1); no longer U2.D11 (PCLKT1_1)
- net GND: now also J5.3 (Pin_3), J5.4 (Pin_4), J8.3 (Pin_3), J8.4 (Pin_4), J9.3 (Pin_3), J9.4 (Pin_4), J10.2 (Pin_2), R15.2, R26.2, R30.2, R59.2, R60.2, R61.2, R62.2, R63.2; no longer J5.10 (Pin_10), J5.9 (Pin_9), J8.10 (Pin_10), J8.9 (Pin_9), J9.10 (Pin_10), J9.9 (Pin_9)
- net PMOD0_1: now also J5.11 (Pin_11), U2.A12 (PT76A); no longer J5.1 (Pin_1), U2.D14 (PT85A)
- net PMOD0_2: now also J5.9 (Pin_9), U2.D12 (GR_PCLK1_0); no longer J5.2 (Pin_2), U2.A14 (PT83A)
- net PMOD0_3: now also J5.7 (Pin_7), U2.A13 (PT76B); no longer J5.3 (Pin_3), U2.D13 (PT80A)
- net PMOD0_4: now also J5.5 (Pin_5), U2.D13 (PT80A); no longer J5.4 (Pin_4), U2.B13 (PT78A)
- net PMOD0_5: now also J5.12 (Pin_12), U2.B12 (PCLKT1_0); no longer J5.5 (Pin_5), U2.A12 (PT76A)
- net PMOD0_6: now also J5.10 (Pin_10), U2.C12 (PCLKC1_0); no longer J5.6 (Pin_6), U2.D12 (GR_PCLK1_0)
- net PMOD0_7: now also J5.8 (Pin_8), U2.B13 (PT78A); no longer J5.7 (Pin_7), U2.B12 (PCLKT1_0)
- net PMOD0_8: now also J5.6 (Pin_6), U2.C13 (PT78B); no longer J5.8 (Pin_8), U2.B15 (PT105A)
- net PMOD1_1: now also J8.11 (Pin_11), U2.A14 (PT83A); no longer J8.1 (Pin_1), U2.C14 (PT83B)
- net PMOD1_2: now also J8.9 (Pin_9), U2.B15 (PT105A); no longer J8.2 (Pin_2), U2.E13 (PT80B)
- net PMOD1_3: now also J8.7 (Pin_7), U2.C15 (PT105B); no longer J8.3 (Pin_3), U2.C13 (PT78B)
- net PMOD1_4: now also J8.5 (Pin_5), U2.B16 (PT110B); no longer J8.4 (Pin_4), U2.A13 (PT76B)
- net PMOD1_5: now also J8.12 (Pin_12), U2.C14 (PT83B); no longer J8.5 (Pin_5), U2.E12 (GR_PCLK1_1)
- net PMOD1_6: now also J8.10 (Pin_10), U2.D15 (PT107A); no longer J8.6 (Pin_6), U2.C12 (PCLKC1_0)
- net PMOD1_7: now also J8.8 (Pin_8), U2.A16 (PT110A); no longer J8.7 (Pin_7), U2.E11 (PCLKC1_1)
- net PMOD1_8: now also J8.6 (Pin_6), U2.C16 (PT112A); no longer J8.8 (Pin_8), U2.E14 (PT85B)
- net PMOD2_1: now also J9.11 (Pin_11), U2.A17 (PT116A); no longer J9.1 (Pin_1), U2.A18 (PT119A)
- net PMOD2_2: now also J9.9 (Pin_9), U2.C17 (PT114B); no longer J9.2 (Pin_2), U2.A17 (PT116A)
- net PMOD2_3: now also J9.7 (Pin_7), U2.B18 (PT116B); no longer J9.3 (Pin_3), U2.B17 (PT114A)
- net PMOD2_4: now also J9.5 (Pin_5), U2.B20 (PT121B); no longer J9.4 (Pin_4), U2.C16 (PT112A)
- net PMOD2_5: now also J9.12 (Pin_12), U2.B17 (PT114A); no longer J9.5 (Pin_5), U2.A16 (PT110A)
- net PMOD2_6: now also J9.10 (Pin_10), U2.A18 (PT119A); no longer J9.6 (Pin_6), U2.D15 (PT107A)
- net PMOD2_7: now also J9.8 (Pin_8), U2.A19 (PT121A); no longer J9.7 (Pin_7), U2.C15 (PT105B)
- net PMOD2_8: now also J9.6 (Pin_6), U2.B19 (PT119B); no longer J9.8 (Pin_8), U2.A19 (PT121A)
- removed net BANK0: U2.A10 (PCLKT0_1), U2.A11 (PCLKC0_1), U2.A6 (PT4A), U2.A7 (PT18A), U2.A8 (PT18B), U2.A9 (GR_PCLK0_1), U2.B10 (GR_PCLK0_0), U2.B11 (PCLKT0_0), U2.B6 (PT4B), U2.B8 (PT15B), U2.B9 (PT58A), U2.C10 (PT58B), U2.C11 (PCLKC0_0), U2.C6 (PT11A), U2.C7 (PT11B), U2.C8 (PT15A), U2.C9 (PT54A), U2.D10 (PT56A), U2.D6 (PT6B), U2.D7 (PT9B), U2.D8 (PT13B), U2.D9 (PT20A), U2.E10 (PT56B), U2.E6 (PT6A), U2.E7 (PT9A), U2.E8 (PT13A), U2.E9 (PT20B)
- removed net BANK7: U2.A2 (PL35A), U2.A3 (PL14C), U2.A4 (PL11A), U2.A5 (PL11B), U2.B1 (PL35B), U2.B2 (VREF1_7), U2.B3 (PL14D), U2.B4 (PL14B), U2.B5 (PL11C), U2.C1 (PL38A), U2.C2 (PL35D), U2.C3 (PL17C), U2.C4 (PL14A), U2.C5 (PL11D), U2.D1 (PL38B), U2.D2 (PL38C), U2.D3 (PL17D), U2.D5 (PL17B), U2.E1 (PL38D), U2.E2 (PCLKC7_0), U2.E3 (PL20B), U2.E4 (PL17A), U2.E5 (PL20C), U2.F2 (PCLKT7_0), U2.F3 (PCLKC7_1), U2.F4 (PL20A), U2.F5 (PL20D), U2.G3 (PCLKT7_1), U2.G5 (PL41B), U2.H3 (PL41D), U2.H4 (GR_PCLK7_1), U2.H5 (GR_PCLK7_0)
- removed net PMOD0_VCC: J5.11 (Pin_11), J5.12 (Pin_12)
- removed net PMOD1_VCC: J8.11 (Pin_11), J8.12 (Pin_12)
- removed net PMOD2_VCC: J9.11 (Pin_11), J9.12 (Pin_12)
- new net: D3.1 (K), R15.1
- new net: D4.1 (K), R26.1
- new net: D5.1 (K), R30.1
- new net: D6.1 (K), R59.1
- new net: D7.1 (K), R60.1
- new net: D8.1 (K), R61.1
- new net: D9.1 (K), R62.1
- new net: D10.1 (K), R63.1
- new net WIDE_1: J4.1 (Pin_1), U2.F3 (PCLKC7_1)
- new net WIDE_10: J4.10 (Pin_10), U2.B2 (VREF1_7)
- new net WIDE_11: J4.11 (Pin_11), U2.A3 (PL14C)
- new net WIDE_12: J4.12 (Pin_12), U2.D2 (PL38C)
- new net WIDE_13: J4.13 (Pin_13), U2.C3 (PL17C)
- new net WIDE_14: J4.14 (Pin_14), U2.B3 (PL14D)
- new net WIDE_15: J4.15 (Pin_15), U2.A4 (PL11A)
- new net WIDE_16: J4.16 (Pin_16), U2.D3 (PL17D)
- new net WIDE_17: J4.17 (Pin_17), U2.C4 (PL14A)
- new net WIDE_18: J4.18 (Pin_18), U2.B4 (PL14B)
- new net WIDE_19: J4.19 (Pin_19), U2.A5 (PL11B)
- new net WIDE_2: J4.2 (Pin_2), U2.F2 (PCLKT7_0)
- new net WIDE_20: J4.20 (Pin_20), U2.E4 (PL17A)
- new net WIDE_21: J4.21 (Pin_21), U2.C5 (PL11D)
- new net WIDE_22: J4.22 (Pin_22), U2.B5 (PL11C)
- new net WIDE_23: J4.23 (Pin_23), U2.A6 (PT4A)
- new net WIDE_24: J4.24 (Pin_24), U2.D5 (PL17B)
- new net WIDE_25: J4.25 (Pin_25), U2.C6 (PT11A)
- new net WIDE_26: J4.26 (Pin_26), U2.B6 (PT4B)
- new net WIDE_27: J4.27 (Pin_27), U2.C7 (PT11B)
- new net WIDE_28: J4.28 (Pin_28), U2.A7 (PT18A)
- new net WIDE_29: J4.29 (Pin_29), U2.B8 (PT15B)
- new net WIDE_3: J4.3 (Pin_3), U2.E2 (PCLKC7_0)
- new net WIDE_30: J4.30 (Pin_30), U2.A8 (PT18B)
- new net WIDE_31: J4.31 (Pin_31), U2.A9 (GR_PCLK0_1)
- new net WIDE_32: J4.32 (Pin_32), U2.C8 (PT15A)
- new net WIDE_33: D3.2 (A), J4.33 (Pin_33), U2.C9 (PT54A)
- new net WIDE_34: D4.2 (A), J4.34 (Pin_34), U2.B9 (PT58A)
- new net WIDE_35: D5.2 (A), J4.35 (Pin_35), U2.B10 (GR_PCLK0_0)
- new net WIDE_36: D6.2 (A), J4.36 (Pin_36), U2.A10 (PCLKT0_1)
- new net WIDE_37: D7.2 (A), J4.37 (Pin_37), U2.A11 (PCLKC0_1)
- new net WIDE_38: D8.2 (A), J4.38 (Pin_38), U2.C10 (PT58B)
- new net WIDE_39: D9.2 (A), J4.39 (Pin_39), U2.B11 (PCLKT0_0)
- new net WIDE_4: J4.4 (Pin_4), U2.E1 (PL38D)
- new net WIDE_40: D10.2 (A), J4.40 (Pin_40), U2.C11 (PCLKC0_0)
- new net WIDE_5: J4.5 (Pin_5), U2.C1 (PL38A)
- new net WIDE_6: J4.6 (Pin_6), U2.D1 (PL38B)
- new net WIDE_7: J4.7 (Pin_7), U2.A2 (PL35A)
- new net WIDE_8: J4.8 (Pin_8), U2.B1 (PL35B)
- new net WIDE_9: J4.9 (Pin_9), U2.C2 (PL35D)
- no-connect marks 57 -> 75
Other:
- note added: "TODO: Add 1V8 rail"
- moved on the sheet: J5, J8, J9, U2A, U2B, U2F

Commit message: Final RevA
Parts:
- added C6: 100n, Capacitor_SMD:C_0603_1608Metric, symbol Device:C_Small
- added J11: Conn_02x04_Odd_Even, Connector_PinHeader_2.54mm:PinHeader_2x04_P2.54mm_Vertical_SMD, symbol Connector_Generic:Conn_02x04_Odd_Even
Connections:
- net +2V5: now also C6.1
- net +3V3: now also J11.2 (Pin_2)
- net FLASH_CSn: now also J11.1 (Pin_1)
- net FLASH_HOLDn: now also J11.4 (Pin_4)
- net FLASH_MISO: now also J11.3 (Pin_3)
- net FLASH_MOSI: now also J11.8 (Pin_8)
- net FLASH_SCK: now also J11.6 (Pin_6)
- net FLASH_WPn: now also J11.5 (Pin_5)
- net FT_GPIO1: now also U2.G5 (PL41B)
- net GND: now also C6.2, J11.7 (Pin_7)
- no-connect marks 75 -> 93
Changed lines of the file:
@@
 	21550 13150 21650 13250
 Entry Wire Line
-	21550 13650 21650 13750
-Entry Wire Line
 	21550 13850 21650 13950
 Entry Wire Line
@@
 Entry Wire Line
 	18850 13250 18950 13150
-Entry Wire Line
-	18850 13450 18950 13350
-Entry Wire Line
-	18850 13550 18950 13450
-Entry Wire Line
-	18850 13750 18950 13650
 Entry Wire Line
 	18850 13950 18950 13850
@@
 	18500 1900 18500 2000
 Connection ~ 18800 1900
-Wire Wire Line
-	18800 1900 19100 1900
 $Comp
 L power:+2V5 #PWR081
@@
 	10150 13150 10250 13050
 Entry Wire Line
-	10150 13250 10250 13150
-Entry Wire Line
-	10150 13350 10250 13250
-Entry Wire Line
-	10150 13450 10250 13350
-Entry Wire Line
 	10150 13550 10250 13450
-Entry Wire Line
-	10150 13650 10250 13550
-Entry Wire Line
-	10150 13750 10250 13650
-Entry Wire Line
-	10150 13850 10250 13750
 Wire Wire Line
 	10850 12250 10250 12250
@@
 	10850 13050 10250 13050
 Wire Wire Line
-	10850 13150 10250 13150
-Wire Wire Line
-	10850 13250 10250 13250
-Wire Wire Line
-	10850 13350 10250 13350
-Wire Wire Line
 	10850 13450 10250 13450
-Wire Wire Line
-	10850 13550 10250 13550
-Wire Wire Line
-	10850 13650 10250 13650
-Wire Wire Line
-	10850 13750 10250 13750
 Text Label 19550 12650 2    50   ~ 0
 RAM_DQ0
@@
 	21050 13150 21550 13150
 Wire Wire Line
-	21050 13650 21550 13650
-Wire Wire Line
 	21050 13850 21550 13850
 Wire Wire Line
@@
 Wire Wire Line
 	19550 13150 18950 13150
-Wire Wire Line
-	19550 13350 18950 13350
-Wire Wire Line
-	19550 13450 18950 13450
-Wire Wire Line
-	19550 13650 18950 13650
 Wire Wire Line
 	19550 13850 18950 13850
@@
 	12350 12950 12850 12950
 Wire Wire Line
-	12350 13050 12850 13050
-Wire Wire Line
 	12350 13450 12850 13450
 Entry Wire Line
@@
 Entry Wire Line
 	12850 12950 12950 13050
-Entry Wire Line
-	12850 13050 12950 13150
 NoConn ~ 12350 13150
 NoConn ~ 12350 13250
@@
 Text Label 2350 8850 0    50   ~ 0
 998-MIC5504-1.8YM5TR
+$Comp
+L Connector_Generic:Conn_02x04_Odd_Even J11
+U 1 1 63303D58
+P 5400 11550
+F 0 "J11" H 5450 11867 50  0000 C CNN
+F 1 "Conn_02x04_Odd_Even" H 5450 11776 50  0000 C CNN
+F 2 "Connector_PinHeader_2.54mm:PinHeader_2x04_P2.54mm_Vertical_SMD" H 5400 11550 50  0001 C CNN
+F 3 "~" H 5400 11550 50  0001 C CNN
+	1    5400 11550
+	1    0    0    -1
+$EndComp
+$Comp
+L power:+3V3 #PWR0129
+U 1 1 63303EDA
+P 5700 11450
+F 0 "#PWR0129" H 5700 11300 50  0001 C CNN
+F 1 "+3V3" V 5700 11650 50  0000 C CNN
+F 2 "" H 5700 11450 50  0001 C CNN
+F 3 "" H 5700 11450 50  0001 C CNN
+	1    5700 11450
+	0    1    1    0
+$EndComp
+Text Label 5200 11450 2    50   ~ 0
+FLASH_CSn
+Text Label 5200 11550 2    50   ~ 0
+FLASH_MISO
+Text Label 5200 11650 2    50   ~ 0
+FLASH_WPn
+$Comp
+L power:GND #PWR0130
+U 1 1 6330928B
+P 5200 11750
+F 0 "#PWR0130" H 5200 11500 50  0001 C CNN
+F 1 "GND" V 5200 11550 50  0000 C CNN
+F 2 "" H 5200 11750 50  0001 C CNN
+F 3 "" H 5200 11750 50  0001 C CNN
+	1    5200 11750
+	0    1    1    0
+$EndComp
+Text Label 5700 11550 0    50   ~ 0
+FLASH_HOLDn
+Text Label 5700 11650 0    50   ~ 0
+FLASH_SCK
+Text Label 5700 11750 0    50   ~ 0
+FLASH_MOSI
+NoConn ~ 13200 15850
+NoConn ~ 13200 15950
+NoConn ~ 13200 16450
+NoConn ~ 13200 16550
+NoConn ~ 14700 16450
+NoConn ~ 14700 15950
+NoConn ~ 14700 15850
+NoConn ~ 10850 13150
+NoConn ~ 10850 13250
+NoConn ~ 10850 13350
+NoConn ~ 10850 13550
+NoConn ~ 10850 13650
+NoConn ~ 10850 13750
+NoConn ~ 12350 13050
+NoConn ~ 19550 13350
+NoConn ~ 19550 13450
+NoConn ~ 19550 13650
+NoConn ~ 21050 13650
+$Comp
+L power:PWR_FLAG #FLG0101
+U 1 1 646CD89C
+P 5800 1650
+F 0 "#FLG0101" H 5800 1725 50  0001 C CNN
+F 1 "PWR_FLAG" H 5800 1824 50  0001 C CNN
+F 2 "" H 5800 1650 50  0001 C CNN
+F 3 "~" H 5800 1650 50  0001 C CNN
+	1    5800 1650
+	-1   0    0    1
+$EndComp
+Wire Wire Line
+	5800 1600 5800 1650
+Text GLabel 14700 16550 2    50   Input ~ 0
+FT_GPIO1
+$Comp
+L power:PWR_FLAG #FLG0102
+U 1 1 64DA45CA
+P 6100 1650
+F 0 "#FLG0102" H 6100 1725 50  0001 C CNN
+F 1 "PWR_FLAG" H 6100 1824 50  0001 C CNN
+F 2 "" H 6100 1650 50  0001 C CNN
+F 3 "~" H 6100 1650 50  0001 C CNN
+	1    6100 1650
+	-1   0    0    1
+$EndComp
+Wire Wire Line
+	6100 1600 6100 1650
+$Comp
+L power:+3V3 #PWR0131
+U 1 1 64DA45D1
+P 6100 1600
+F 0 "#PWR0131" H 6100 1450 50  0001 C CNN
+F 1 "+3V3" H 6115 1773 50  0000 C CNN
+F 2 "" H 6100 1600 50  0001 C CNN
+F 3 "" H 6100 1600 50  0001 C CNN
+	1    6100 1600
+	1    0    0    -1
+$EndComp
+$Comp
+L power:PWR_FLAG #FLG0103
+U 1 1 64E9D048
+P 6400 1650
+F 0 "#FLG0103" H 6400 1725 50  0001 C CNN
+F 1 "PWR_FLAG" H 6400 1824 50  0001 C CNN
+F 2 "" H 6400 1650 50  0001 C CNN
+F 3 "~" H 6400 1650 50  0001 C CNN
+	1    6400 1650
+	-1   0    0    1
+$EndComp
+Wire Wire Line
+	6400 1600 6400 1650
+$Comp
+L power:PWR_FLAG #FLG0104
+U 1 1 64F9621E
+P 6700 1650
+F 0 "#FLG0104" H 6700 1725 50  0001 C CNN
+F 1 "PWR_FLAG" H 6700 1824 50  0001 C CNN
+F 2 "" H 6700 1650 50  0001 C CNN
+F 3 "~" H 6700 1650 50  0001 C CNN
+	1    6700 1650
+	-1   0    0    1
+$EndComp
+Wire Wire Line
+	6700 1600 6700 1650
+$Comp
+L power:+5V #PWR0132
+U 1 1 6508FE0B
+P 5800 1600
+F 0 "#PWR0132" H 5800 1450 50  0001 C CNN
+F 1 "+5V" H 5815 1773 50  0000 C CNN
+F 2 "" H 5800 1600 50  0001 C CNN
+F 3 "" H 5800 1600 50  0001 C CNN
+	1    5800 1600
+	1    0    0    -1
+$EndComp
+$Comp
+L power:+2V5 #PWR0133
+U 1 1 650908E9
+P 6400 1600
+F 0 "#PWR0133" H 6400 1450 50  0001 C CNN
+F 1 "+2V5" H 6415 1773 50  0000 C CNN
+F 2 "" H 6400 1600 50  0001 C CNN
+F 3 "" H 6400 1600 50  0001 C CNN
+	1    6400 1600
+	1    0    0    -1
+$EndComp
+$Comp
+L power:+1V1 #PWR0134
+U 1 1 65090C13
+P 6700 1600
+F 0 "#PWR0134" H 6700 1450 50  0001 C CNN
+F 1 "+1V1" H 6715 1773 50  0000 C CNN
+F 2 "" H 6700 1600 50  0001 C CNN
+F 3 "" H 6700 1600 50  0001 C CNN
+	1    6700 1600
+	1    0    0    -1
+$EndComp
+$Comp
+L Device:C_Small C6
+U 1 1 653841FA
+P 19100 2100
+F 0 "C6" H 19150 2200 50  0000 L CNN
+F 1 "100n" H 19150 2000 50  0000 L CNN
+F 2 "Capacitor_SMD:C_0603_1608Metric" H 19100 2100 50  0001 C CNN
+F 3 "~" H 19100 2100 50  0001 C CNN
+	1    19100 2100
+	1    0    0    -1
+$EndComp
+Wire Wire Line
+	18800 1900 19100 1900
+Wire Wire Line
+	19100 2000 19100 1900
+$Comp
+L power:GND #PWR0135
+U 1 1 65578ED2
+P 19100 2300
+F 0 "#PWR0135" H 19100 2050 50  0001 C CNN
+F 1 "GND" H 19105 2127 50  0000 C CNN
+F 2 "" H 19100 2300 50  0001 C CNN
+F 3 "" H 19100 2300 50  0001 C CNN
+	1    19100 2300
+	1    0    0    -1
+$EndComp
+Wire Wire Line
+	19100 2300 19100 2200
 Wire Bus Line
 	18150 9200 21550 9200
@@
 	12700 7100 12700 9100
 Wire Bus Line
-	18850 12750 18850 14200
+	12950 12350 12950 14200
 Wire Bus Line
 	21650 12550 21650 14200
 Wire Bus Line
-	12950 12350 12950 14200
+	18850 12750 18850 14200
+Wire Bus Line
+	10150 12350 10150 14200
+Wire Bus Line
+	19050 6500 19050 9100
+Wire Bus Line
+	14350 11350 14350 14200
+Wire Bus Line
+	17650 11350 17650 14200
 Wire Bus Line
 	21650 6500 21650 9100
 Wire Bus Line
-	10150 12350 10150 14200
-Wire Bus Line
-	17650 11350 17650 14200
-Wire Bus Line
-	14350 11350 14350 14200
-Wire Bus Line
-	19050 6500 19050 9100
-Wire Bus Line
 	18050 6500 18050 9100
