File: Kilsyth.sch (KiCad schematic (older format))
At the start: 167 parts, among them J1 Conn_JTAG, J10 Conn_02x01, J11 Conn_02x04_Odd_Even, J2 DX07S024JJ2, J3 USB_B_Micro, J4 Conn_02x20_Odd_Even, J5 Conn_02x06_Odd_Even, J6 PUSB3FR4Z, J7 PUSB3FR4Z, J8 Conn_02x06_Odd_Even, J9 Conn_02x06_Odd_Even, SW1 SW_Push, U1 DSC6001CI2A-016.0000T, U2 LFE5U-85F-6BG381C, U3 TPS65261, U5 IS25LP128F-JBLE, U6 FT600Q, U7 AS4C32M16SB, Y1 30MHz ±20ppm

Commit message: Last minute changes
Parts:
- added J12: Conn_02x04_Odd_Even, Connector_PinHeader_2.54mm:PinHeader_2x04_P2.54mm_Vertical_SMD, symbol Connector_Generic:Conn_02x04_Odd_Even
Connections:
- net +3V3: now also J12.2 (Pin_2), J12.4 (Pin_4), J12.6 (Pin_6), J12.8 (Pin_8)
- net GND: now also J12.1 (Pin_1), J12.3 (Pin_3), J12.5 (Pin_5), J12.7 (Pin_7)
Changed lines of the file:
@@
 Wire Wire Line
 	19100 2300 19100 2200
+$Comp
+L Connector_Generic:Conn_02x04_Odd_Even J12
+U 1 1 5C1DB034
+P 5800 2250
+F 0 "J12" H 5850 2567 50  0000 C CNN
+F 1 "Conn_02x04_Odd_Even" H 5850 2476 50  0000 C CNN
+F 2 "Connector_PinHeader_2.54mm:PinHeader_2x04_P2.54mm_Vertical_SMD" H 5800 2250 50  0001 C CNN
+F 3 "~" H 5800 2250 50  0001 C CNN
+	1    5800 2250
+	1    0    0    -1
+$EndComp
+$Comp
+L power:+3V3 #PWR0136
+U 1 1 5C1DBB26
+P 6100 2150
+F 0 "#PWR0136" H 6100 2000 50  0001 C CNN
+F 1 "+3V3" V 6100 2350 50  0000 C CNN
+F 2 "" H 6100 2150 50  0001 C CNN
+F 3 "" H 6100 2150 50  0001 C CNN
+	1    6100 2150
+	0    1    1    0
+$EndComp
+$Comp
+L power:+3V3 #PWR0137
+U 1 1 5C1DC96C
+P 6100 2250
+F 0 "#PWR0137" H 6100 2100 50  0001 C CNN
+F 1 "+3V3" V 6100 2450 50  0000 C CNN
+F 2 "" H 6100 2250 50  0001 C CNN
+F 3 "" H 6100 2250 50  0001 C CNN
+	1    6100 2250
+	0    1    1    0
+$EndComp
+$Comp
+L power:+3V3 #PWR0138
+U 1 1 5C1DCADF
+P 6100 2350
+F 0 "#PWR0138" H 6100 2200 50  0001 C CNN
+F 1 "+3V3" V 6100 2550 50  0000 C CNN
+F 2 "" H 6100 2350 50  0001 C CNN
+F 3 "" H 6100 2350 50  0001 C CNN
+	1    6100 2350
+	0    1    1    0
+$EndComp
+$Comp
+L power:+3V3 #PWR0139
+U 1 1 5C1DCC52
+P 6100 2450
+F 0 "#PWR0139" H 6100 2300 50  0001 C CNN
+F 1 "+3V3" V 6100 2650 50  0000 C CNN
+F 2 "" H 6100 2450 50  0001 C CNN
+F 3 "" H 6100 2450 50  0001 C CNN
+	1    6100 2450
+	0    1    1    0
+$EndComp
+$Comp
+L power:GND #PWR0140
+U 1 1 5C1DCDC5
+P 5600 2150
+F 0 "#PWR0140" H 5600 1900 50  0001 C CNN
+F 1 "GND" V 5605 1977 50  0000 C CNN
+F 2 "" H 5600 2150 50  0001 C CNN
+F 3 "" H 5600 2150 50  0001 C CNN
+	1    5600 2150
+	0    1    1    0
+$EndComp
+$Comp
+L power:GND #PWR0141
+U 1 1 5C1DD91F
+P 5600 2250
+F 0 "#PWR0141" H 5600 2000 50  0001 C CNN
+F 1 "GND" V 5605 2077 50  0000 C CNN
+F 2 "" H 5600 2250 50  0001 C CNN
+F 3 "" H 5600 2250 50  0001 C CNN
+	1    5600 2250
+	0    1    1    0
+$EndComp
+$Comp
+L power:GND #PWR0142
+U 1 1 5C1DDA92
+P 5600 2350
+F 0 "#PWR0142" H 5600 2100 50  0001 C CNN
+F 1 "GND" V 5605 2177 50  0000 C CNN
+F 2 "" H 5600 2350 50  0001 C CNN
+F 3 "" H 5600 2350 50  0001 C CNN
+	1    5600 2350
+	0    1    1    0
+$EndComp
+$Comp
+L power:GND #PWR0143
+U 1 1 5C1DDC05
+P 5600 2450
+F 0 "#PWR0143" H 5600 2200 50  0001 C CNN
+F 1 "GND" V 5605 2277 50  0000 C CNN
+F 2 "" H 5600 2450 50  0001 C CNN
+F 3 "" H 5600 2450 50  0001 C CNN
+	1    5600 2450
+	0    1    1    0
+$EndComp
 Wire Bus Line
 	18150 9200 21550 9200
