File: Kilsyth.kicad_pcb (KiCad board)
At the start: 2 copper layers, 1 part, among them U2 LFE5U-85F-6BG381C

Commit message: More progress
Parts:
- added C1: 1u, Capacitor_SMD:C_0603_1608Metric, F.Cu at (103.8, 101.2)
- added C10: 22p, Capacitor_SMD:C_0603_1608Metric, F.Cu at (103.8, 102.7)
- added C11: 22p, Capacitor_SMD:C_0603_1608Metric, F.Cu at (116.9, 89.9)
- added C12: 22p, Capacitor_SMD:C_0603_1608Metric, F.Cu at (98.4, 107.7)
- added C13: 47n, Capacitor_SMD:C_0603_1608Metric, F.Cu at (106.8, 99.7)
- added C14: 47n, Capacitor_SMD:C_0603_1608Metric, F.Cu at (116.9, 88.4)
- added C15: 47n, Capacitor_SMD:C_0603_1608Metric, F.Cu at (107.9, 92.1)
- added C16: 3.3n, Capacitor_SMD:C_0603_1608Metric, F.Cu at (107.9, 95.1)
- added C17: 3.3n, Capacitor_SMD:C_0603_1608Metric, F.Cu at (100.7, 101.2)
- added C18: 3.3n, Capacitor_SMD:C_0603_1608Metric, F.Cu at (100.7, 98.2)
- added C19: 22p, Capacitor_SMD:C_0603_1608Metric, F.Cu at (104.7, 96.7)
- added C2: 10u, Capacitor_SMD:C_0603_1608Metric, F.Cu at (110.9, 94.4)
- added C20: 22p, Capacitor_SMD:C_0603_1608Metric, F.Cu at (113.9, 88.4)
- added C21: 22p, Capacitor_SMD:C_0603_1608Metric, F.Cu at (107.9, 93.6)
- added C22: 22u, Capacitor_SMD:C_0603_1608Metric, F.Cu at (103.8, 98.2)
- added C23: 22u, Capacitor_SMD:C_0603_1608Metric, F.Cu at (116.8, 85.4)
- added C24: 22u, Capacitor_SMD:C_0603_1608Metric, F.Cu at (95.4, 106.2)
- added C25: 22u, Capacitor_SMD:C_0603_1608Metric, F.Cu at (94.7, 103.2)
- added C26: 100n, Capacitor_SMD:C_0603_1608Metric, F.Cu at (113.9, 89.9)
- added C27: 100n, Capacitor_SMD:C_0603_1608Metric, F.Cu at (116.8, 86.9)
- added C28: 100n, Capacitor_SMD:C_0603_1608Metric, F.Cu at (100.7, 102.7)
- added C29: 18p, Capacitor_SMD:C_0603_1608Metric, F.Cu at (110.9, 92.9)
- added C3: 10u, Capacitor_SMD:C_0603_1608Metric, F.Cu at (113.9, 91.4)
- added C30: 18p, Capacitor_SMD:C_0603_1608Metric, F.Cu at (98.4, 106.2)
- added C31: 100n, Capacitor_SMD:C_0603_1608Metric, F.Cu at (107.9, 96.6)
- added C32: 4u7, Capacitor_SMD:C_0603_1608Metric, F.Cu at (100.7, 104.2)
- added C4: 10u, Capacitor_SMD:C_0603_1608Metric, F.Cu at (117.7, 80.9)
- added C5: 10u, Capacitor_SMD:C_0603_1608Metric, F.Cu at (104.9, 93.6)
- added C6: 22u, Capacitor_SMD:C_0603_1608Metric, F.Cu at (113.8, 85.4)
- added C7: 10n, Capacitor_SMD:C_0603_1608Metric, F.Cu at (107.9, 90.5)
- added C8: 10n, Capacitor_SMD:C_0603_1608Metric, F.Cu at (113.8, 86.9)
- added C9: 10n, Capacitor_SMD:C_0603_1608Metric, F.Cu at (113.9, 92.9)
- added D1: LED, LED_SMD:LED_0603_1608Metric, F.Cu at (71.5, 107.7)
- added FB1: Ferrite_Bead_Small, Inductor_SMD:L_0603_1608Metric, F.Cu at (95.4, 107.7)
- added J2: USB_B_Micro, Connector_USB:USB_Micro-B_Molex_47346-0001, F.Cu at (52.6, 78.0)
- added J3: USB_C_Receptacle, JAE-USB-C:USBC_DX07S024JJ2R1300, F.Cu at (55.0, 90.2)
- added J4: Conn_JTAG, Connector_PinSocket_2.54mm:PinSocket_2x03_P2.54mm_Vertical_SMD, F.Cu at (83.0, 100.1)
- added J5: PUSB3FR4Z, PUSB3FR4Z:PUSB3FR4Z, F.Cu at (61.2, 97.2)
- added L1: 2.2u, Inductor_SMD:L_0603_1608Metric, F.Cu at (110.9, 91.4)
- added L2: 2.2u, Inductor_SMD:L_0603_1608Metric, F.Cu at (117.7, 83.9)
- added L3: 2.2u, Inductor_SMD:L_0603_1608Metric, F.Cu at (97.7, 104.7)
- added R1: 73.2K, Resistor_SMD:R_0603_1608Metric, F.Cu at (104.9, 92.1)
- added R10: 15K, Resistor_SMD:R_0603_1608Metric, F.Cu at (107.8, 84.5)
- added R11: 4.7K, Resistor_SMD:R_0603_1608Metric, F.Cu at (107.8, 86.0)
- added R12: 15K, Resistor_SMD:R_0603_1608Metric, F.Cu at (114.7, 80.9)
- added R13: 3.3K, Resistor_SMD:R_0603_1608Metric, F.Cu at (97.7, 98.7)
- added R14: 0R, Resistor_SMD:R_0603_1608Metric, F.Cu at (97.7, 101.7)
- added R15: 0R, Resistor_SMD:R_0603_1608Metric, F.Cu at (117.7, 82.4)
- added R16: 0R, Resistor_SMD:R_0603_1608Metric, F.Cu at (110.9, 89.9)
- added R17: 0R, Resistor_SMD:R_0603_1608Metric, F.Cu at (110.8, 86.9)
- added R18: 5K1, Resistor_SMD:R_0603_1608Metric, F.Cu at (104.9, 95.1)
- added R19: 5K1, Resistor_SMD:R_0603_1608Metric, F.Cu at (110.9, 88.4)
- added R2: 2K, Resistor_SMD:R_0603_1608Metric, F.Cu at (98.9, 89.1)
- added R20: 0R, Resistor_SMD:R_0603_1608Metric, F.Cu at (106.8, 98.2)
- added R21: 0R, Resistor_SMD:R_0603_1608Metric, F.Cu at (86.4, 107.4)
- added R22: 0R, Resistor_SMD:R_0603_1608Metric, F.Cu at (92.4, 107.4)
- added R23: 0R, Resistor_SMD:R_0603_1608Metric, F.Cu at (114.7, 83.9)
- added R24: 1.6K, Resistor_SMD:R_0603_1608Metric, F.Cu at (94.7, 104.7)
- added R25: 10K, Resistor_SMD:R_0603_1608Metric, F.Cu at (98.7, 96.7)
- added R26: 10K, Resistor_SMD:R_0603_1608Metric, F.Cu at (95.6, 95.7)
- added R27: 10K, Resistor_SMD:R_0603_1608Metric, F.Cu at (94.7, 98.7)
- added R28: 0R, Resistor_SMD:R_0603_1608Metric, F.Cu at (98.9, 92.1)
- added R29: 0R, Resistor_SMD:R_0603_1608Metric, F.Cu at (97.7, 103.2)
- added R3: 4.7K, Resistor_SMD:R_0603_1608Metric, F.Cu at (114.7, 82.4)
- added R30: 0R, Resistor_SMD:R_0603_1608Metric, F.Cu at (104.9, 90.6)
- added R31: 0R, Resistor_SMD:R_0603_1608Metric, F.Cu at (100.7, 99.7)
- added R32: 0R, Resistor_SMD:R_0603_1608Metric, F.Cu at (74.5, 107.7)
- added R33: 0R, Resistor_SMD:R_0603_1608Metric, F.Cu at (98.9, 93.6)
- added R34: 0R, Resistor_SMD:R_0603_1608Metric, F.Cu at (101.7, 96.7)
- added R35: 0R, Resistor_SMD:R_0603_1608Metric, F.Cu at (104.9, 89.1)
- added R36: 0R, Resistor_SMD:R_0603_1608Metric, F.Cu at (94.7, 100.2)
- added R37: 0R, Resistor_SMD:R_0603_1608Metric, F.Cu at (98.9, 90.6)
- added R38: 0R, Resistor_SMD:R_0603_1608Metric, F.Cu at (98.9, 95.1)
- added R39: 0R, Resistor_SMD:R_0603_1608Metric, F.Cu at (101.9, 92.1)
- added R4: 4.7K, Resistor_SMD:R_0603_1608Metric, F.Cu at (101.9, 93.6)
- added R40: 0R, Resistor_SMD:R_0603_1608Metric, F.Cu at (95.6, 97.2)
- added R41: 0R, Resistor_SMD:R_0603_1608Metric, F.Cu at (101.9, 90.6)
- added R42: 0R, Resistor_SMD:R_0603_1608Metric, F.Cu at (92.6, 97.2)
- added R43: 0R, Resistor_SMD:R_0603_1608Metric, F.Cu at (111.7, 80.9)
- added R44: 0R, Resistor_SMD:R_0603_1608Metric, F.Cu at (80.5, 107.7)
- added R45: 0R, Resistor_SMD:R_0603_1608Metric, F.Cu at (92.6, 95.7)
- added R46: 0R, Resistor_SMD:R_0603_1608Metric, F.Cu at (89.6, 95.7)
- added R47: 0R, Resistor_SMD:R_0603_1608Metric, F.Cu at (89.6, 97.2)
- added R48: 0R, Resistor_SMD:R_0603_1608Metric, F.Cu at (77.5, 107.7)
- added R49: 0R, Resistor_SMD:R_0603_1608Metric, F.Cu at (103.8, 99.7)
- added R5: 20K, Resistor_SMD:R_0603_1608Metric, F.Cu at (97.7, 100.2)
- added R50: 0R, Resistor_SMD:R_0603_1608Metric, F.Cu at (101.9, 89.1)
- added R51: 0R, Resistor_SMD:R_0603_1608Metric, F.Cu at (111.7, 82.4)
- added R52: 1M, Resistor_SMD:R_0603_1608Metric, F.Cu at (89.4, 107.4)
- added R53: 1M, Resistor_SMD:R_0603_1608Metric, F.Cu at (111.7, 83.9)
- added R54: 4k7, Resistor_SMD:R_0603_1608Metric, F.Cu at (107.8, 87.5)
- added R6: 20K, Resistor_SMD:R_0603_1608Metric, F.Cu at (94.7, 101.7)
- added R7: 20K, Resistor_SMD:R_0603_1608Metric, F.Cu at (101.9, 95.1)
- added R8: 15K, Resistor_SMD:R_0603_1608Metric, F.Cu at (107.9, 89.0)
- added R9: 18K, Resistor_SMD:R_0603_1608Metric, F.Cu at (110.8, 85.4)
- added TP1: TestPoint, TestPoint:TestPoint_Pad_D1.0mm, F.Cu at (110.4, 96.2)
- added TP2: TestPoint, TestPoint:TestPoint_Pad_D1.0mm, F.Cu at (106.3, 101.5)
- added TP3: TestPoint, TestPoint:TestPoint_Pad_D1.0mm, F.Cu at (109.3, 98.4)
- added TP4: TestPoint, TestPoint:TestPoint_Pad_D1.0mm, F.Cu at (119.4, 85.7)
- added U1: TPS65261, Package_QFP:LQFP-32_5x5mm_P0.5mm, F.Cu at (102.2, 84.2)
- added U3: LFE5U-85F-6BG381C, lfe5bg381:BGA-381_pitch0.8mm_dia0.4mm, F.Cu at (87.2, 84.2)
- added U4: FT600Q, Package_DFN_QFN:QFN-56-1EP_7x7mm_P0.4mm_EP5.7x5.7mm, F.Cu at (69.8, 91.2)
- added U5: IS25LP128F-JBLE, SOA008-150mil:SOA008-150-208mil, F.Cu at (124.0, 115.4)
- added Y1: 30MHz ±20ppm, Crystal:Crystal_SMD_2016-4Pin_2.0x1.6mm, F.Cu at (101.3, 106.3)
- U2: value LFE5U-85F-6BG381C -> MIC5504-1.8YM5; footprint lfe5bg381:BGA-381_pitch0.8mm_dia0.4mm -> Package_TO_SOT_SMD:SOT-23-5
- moved U2 50.5 mm to (108.2, 81.9)
Other:
- board outline added: 95 x 95 mm

Commit message: WIP
Parts:
- added C33: 100n, Capacitor_SMD:C_0603_1608Metric, F.Cu at (99.5, 61.8)
- added C34: 100n, Capacitor_SMD:C_0603_1608Metric, F.Cu at (97.8, 60.3)
- added C35: 4u7, Capacitor_SMD:C_0603_1608Metric, F.Cu at (96.5, 62.2)
- added C36: 100n, Capacitor_SMD:C_0603_1608Metric, F.Cu at (97.8, 58.8)
- added C37: 100n, Capacitor_SMD:C_0603_1608Metric, F.Cu at (93.5, 62.2)
- added U6: DSC6001CI2A-016.0000T, Crystal:Crystal_SMD_3225-4Pin_3.2x2.5mm, F.Cu at (86.2, 55.4)
- C32: value 4u7 -> 100n
- FB1: value Ferrite_Bead_Small -> Ferrite_Bead
- moved TP2 20.0 mm to (126.2, 100.0)
Connections:
- C32 pad 1: VD10 -> +3V3
- FB1 pad 1: VBUS -> +5V
- FB1 pad 2: VBUS -> +5V
- J2 pad 1: VBUS -> +5V
- J3 pad A4: VBUS -> +5V
- J3 pad A9: VBUS -> +5V
- J3 pad B4: VBUS -> +5V
- J3 pad B9: VBUS -> +5V
- U3 pad B12: Net-(U3-PadB12) -> CLK_16MHz
- U3 pad R2: Net-(U3-PadR2) -> /FLASH_CSn
- U3 pad T2: Net-(U3-PadT2) -> +3V3
- U3 pad T3: Net-(U3-PadT3) -> +3V3
- U3 pad U2: Net-(U3-PadU2) -> +3V3
- U3 pad U3: Net-(U3-PadU3) -> /FLASH_SCK
- U3 pad V2: Net-(U3-PadV2) -> /FLASH_MISO
- U3 pad W1: Net-(U3-PadW1) -> /FLASH_HOLDn
- U3 pad W2: Net-(U3-PadW2) -> /FLASH_MOSI
- U3 pad Y2: Net-(U3-PadY2) -> /FLASH_WPn
- U4 pad 29: VBUS -> +5V
- U5 pad 1: Net-(U5-Pad1) -> /FLASH_CSn
- U5 pad 2: Net-(U5-Pad2) -> /FLASH_MISO
- U5 pad 3: Net-(U5-Pad3) -> /FLASH_WPn
- U5 pad 4: Net-(U5-Pad4) -> GND
- U5 pad 5: Net-(U5-Pad5) -> /FLASH_MOSI
- U5 pad 6: Net-(U5-Pad6) -> /FLASH_SCK
- U5 pad 7: Net-(U5-Pad7) -> /FLASH_HOLDn
- U5 pad 8: Net-(U5-Pad8) -> +3V3
Routing:
- added copper zone on F.Cu, net GND

Commit message: Hmmmm
Parts:
- added C38: 4u7, Capacitor_SMD:C_0603_1608Metric, F.Cu at (16.0, 112.0)
- added C39: 100n, Capacitor_SMD:C_0603_1608Metric, F.Cu at (19.0, 108.9)
- added C40: 100n, Capacitor_SMD:C_0603_1608Metric, F.Cu at (33.7, 94.3)
- added C41: 100n, Capacitor_SMD:C_0603_1608Metric, F.Cu at (37.1, 161.1)
- added C42: 100n, Capacitor_SMD:C_0603_1608Metric, F.Cu at (19.0, 104.4)
- added C43: 4u7, Capacitor_SMD:C_0603_1608Metric, F.Cu at (22.0, 99.9)
- added C44: 100n, Capacitor_SMD:C_0603_1608Metric, F.Cu at (23.0, 134.8)
- added C45: 100n, Capacitor_SMD:C_0603_1608Metric, F.Cu at (23.0, 133.3)
- added C46: 100n, Capacitor_SMD:C_0603_1608Metric, F.Cu at (30.7, 94.3)
- added C47: 10n, Capacitor_SMD:C_0603_1608Metric, F.Cu at (16.0, 110.4)
- added C48: 10n, Capacitor_SMD:C_0603_1608Metric, F.Cu at (33.7, 92.8)
- added C49: 10n, Capacitor_SMD:C_0603_1608Metric, F.Cu at (16.0, 108.9)
- added C50: 100n, Capacitor_SMD:C_0603_1608Metric, F.Cu at (19.0, 107.4)
- added C51: 100n, Capacitor_SMD:C_0603_1608Metric, F.Cu at (22.0, 102.9)
- added C52: 10n, Capacitor_SMD:C_0603_1608Metric, F.Cu at (34.8, 126.1)
- added C53: 10n, Capacitor_SMD:C_0603_1608Metric, F.Cu at (28.0, 97.3)
- added C54: 100n, Capacitor_SMD:C_0603_1608Metric, F.Cu at (25.0, 100.4)
- added C55: 100n, Capacitor_SMD:C_0603_1608Metric, F.Cu at (15.1, 143.1)
- added C56: 10n, Capacitor_SMD:C_0603_1608Metric, F.Cu at (12.1, 146.2)
- added C57: 10n, Capacitor_SMD:C_0603_1608Metric, F.Cu at (20.5, 138.2)
- added C58: 100n, Capacitor_SMD:C_0603_1608Metric, F.Cu at (17.5, 140.0)
- added C59: 10n, Capacitor_SMD:C_0603_1608Metric, F.Cu at (19.0, 105.9)
- added C60: 100n, Capacitor_SMD:C_0603_1608Metric, F.Cu at (25.0, 97.3)
- added C61: 10n, Capacitor_SMD:C_0603_1608Metric, F.Cu at (37.1, 162.6)
- added C62: 100n, Capacitor_SMD:C_0603_1608Metric, F.Cu at (16.0, 107.4)
- added C63: 10n, Capacitor_SMD:C_0603_1608Metric, F.Cu at (12.1, 143.1)
- added C64: 100n, Capacitor_SMD:C_0603_1608Metric, F.Cu at (12.1, 141.6)
- added C65: 10n, Capacitor_SMD:C_0603_1608Metric, F.Cu at (14.5, 140.1)
- added C66: 100n, Capacitor_SMD:C_0603_1608Metric, F.Cu at (17.5, 138.4)
- added C67: 10n, Capacitor_SMD:C_0603_1608Metric, F.Cu at (9.13, 144.7)
- added D2: LED, LED_SMD:LED_0603_1608Metric, F.Cu at (7.34, 104.6)
- added H1: , MountingHole:MountingHole_3.2mm_M3_Pad, F.Cu at (55.0, 55.0)
- added H2: , MountingHole:MountingHole_3.2mm_M3_Pad, F.Cu at (140.0, 55.0)
- added H3: , MountingHole:MountingHole_3.2mm_M3_Pad, F.Cu at (55.0, 125.0)
- added H4: , MountingHole:MountingHole_3.2mm_M3_Pad, F.Cu at (140.0, 125.0)
- added J1: Conn_JTAG, Connector_PinSocket_2.54mm:PinSocket_2x03_P2.54mm_Vertical_SMD, F.Cu at (74.5, 120.0)
- added J6: PUSB3FR4Z, PUSB3FR4Z:PUSB3FR4Z, F.Cu at (67.7, 89.0)
- added J7: PUSB3FR4Z, PUSB3FR4Z:PUSB3FR4Z, F.Cu at (67.7, 91.9)
- added J8: Conn_02x06_Counter_Clockwise, Connector_PinSocket_2.54mm:PinSocket_2x06_P2.54mm_Horizontal, F.Cu at (100.1, 124.5)
- added J9: Conn_02x06_Counter_Clockwise, Connector_PinSocket_2.54mm:PinSocket_2x06_P2.54mm_Horizontal, F.Cu at (118.2, 124.7)
- added R55: 0R, Resistor_SMD:R_0603_1608Metric, F.Cu at (25.9, 53.3)
- added R56: 0R, Resistor_SMD:R_0603_1608Metric, F.Cu at (24.9, 57.3)
- added R57: 0R, Resistor_SMD:R_0603_1608Metric, F.Cu at (23.9, 53.3)
- added R58: 0R, Resistor_SMD:R_0603_1608Metric, F.Cu at (22.9, 57.3)
- added SW1: SW_Push, kilsyth_extra:SmallButton, F.Cu at (64.0, 112.0)
- added TP5: TestPoint, TestPoint:TestPoint_Pad_D1.0mm, F.Cu at (21.5, 107.7)
- added U7: AS4C32M16SB, Package_SO:TSOP-II-54_22.2x10.16mm_P0.8mm, F.Cu at (131.0, 90.0)
- C1: value 1u -> 100n
- C10: value 22p -> 10n
- C13: value 47n -> 22p
- C16: value 3.3n -> 47n
- C19: value 22p -> 3.3n
- C2: value 10u -> 1u
- C22: value 22u -> 22p
- C26: value 100n -> 22u
- C29, C30: value 18p -> 100n
- C32: value 100n -> 4u7
- C33, C34: value 100n -> 18p
- C35: value 4u7 -> 100n
- C6: value 22u -> 10u
- C7: value 10n -> 22u
- J2: value USB_B_Micro -> DX07S024JJ2; footprint Connector_USB:USB_Micro-B_Molex_47346-0001 -> JAE-USB-C:USBC_DX07S024JJ2R1300
- J3: value USB_C_Receptacle -> USB_B_Micro; footprint JAE-USB-C:USBC_DX07S024JJ2R1300 -> Connector_USB:USB_Micro-B_Molex_47346-0001
- J4: value Conn_JTAG -> Conn_02x20_Counter_Clockwise; footprint Connector_PinSocket_2.54mm:PinSocket_2x03_P2.54mm_Vertical_SMD -> Connector_PinHeader_2.54mm:PinHeader_2x20_P2.54mm_Vertical_SMD
- J5: value PUSB3FR4Z -> Conn_02x06_Counter_Clockwise; footprint PUSB3FR4Z:PUSB3FR4Z -> Connector_PinSocket_2.54mm:PinSocket_2x06_P2.54mm_Horizontal
- R1: value 73.2K -> 4.7K
- R10: value 15K -> 18K
- R11: value 4.7K -> 15K
- R12: value 15K -> 4.7K
- R13: value 3.3K -> 15K
- R14: value 0R -> 3.3K
- R16: value 0R -> 2K
- R18, R19: value 5K1 -> 0R
- R2: value 2K -> 73.2K
- R20, R22, R32, R33, R34: value 0R -> 10K
- R23: value 0R -> 1M
- R24: value 1.6K -> 1M
- R25, R26: value 10K -> 5K1
- R27: value 10K -> 0R
- R31: value 0R -> 1.6K
- R4: value 4.7K -> 4k7
- R52, R53: value 1M -> 0R
- R54: value 4k7 -> 0R
- R8: value 15K -> 2K
- R9: value 18K -> 15K
- U1: value TPS65261 -> DSC6001CI2A-016.0000T; footprint Package_QFP:LQFP-32_5x5mm_P0.5mm -> Crystal:Crystal_SMD_3225-4Pin_3.2x2.5mm
- U2: value MIC5504-1.8YM5 -> LFE5U-85F-6BG381C; footprint Package_TO_SOT_SMD:SOT-23-5 -> lfe5bg381:BGA-381_pitch0.8mm_dia0.4mm
- U3: value LFE5U-85F-6BG381C -> TPS65261; footprint lfe5bg381:BGA-381_pitch0.8mm_dia0.4mm -> kilsyth_extra:S-PVQFN-N32
- U4: value FT600Q -> MIC5504-1.8YM5; footprint Package_DFN_QFN:QFN-56-1EP_7x7mm_P0.4mm_EP5.7x5.7mm -> Package_TO_SOT_SMD:SOT-23-5
- U6: value DSC6001CI2A-016.0000T -> FT600Q; footprint Crystal:Crystal_SMD_3225-4Pin_3.2x2.5mm -> kilsyth_extra:QFN-56-1EP_7x7mm_P0.4mm_EP5.7x5.7mm_FIXED
- moved C11 132.7 mm to (-15.0, 75.3)
- moved R2 132.0 mm to (-27.7, 51.5)
- moved C22 131.5 mm to (-27.6, 91.4)
- moved C13 129.3 mm to (-22.5, 99.1)
- moved C8 128.9 mm to (-14.8, 78.9)
- moved C10 127.4 mm to (-23.1, 90.8)
- moved R13 125.7 mm to (-27.9, 94.6)
- moved C36 125.5 mm to (9.13, 147.7)
- moved R14 125.3 mm to (-27.5, 98.9)
- moved L2 125.2 mm to (9.13, 146.2)
- moved C14 123.8 mm to (9.13, 149.2)
- moved C35 118.0 mm to (12.1, 144.7)
- moved C6 116.7 mm to (15.1, 147.7)
- moved U3 116.1 mm to (-27.9, 68.9)
- moved R11 114.0 mm to (9.13, 143.1)
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Connections:
- C1 pad 1: Net-(C1-Pad1) -> +3V3
- C13 pad 2: Net-(C13-Pad2) -> GND
- C16 pad 2: GND -> Net-(C16-Pad2)
- C19 pad 2: Net-(C19-Pad2) -> GND
- C2 pad 1: +5V -> Net-(C2-Pad1)
- C22 pad 1: Net-(C19-Pad1) -> Net-(C22-Pad1)
- C22 pad 2: GND -> Net-(C22-Pad2)
- C25 pad 1: Net-(C19-Pad1) -> Net-(C22-Pad1)
- C26 pad 1: Net-(C26-Pad1) -> Net-(C20-Pad1)
- C26 pad 2: /FT_TODN -> GND
- C27 pad 1: Net-(C27-Pad1) -> +3V3
- C27 pad 2: /FT_TODP -> GND
- C29 pad 1: GND -> Net-(C29-Pad1)
- C29 pad 2: Net-(C29-Pad2) -> GND
- C30 pad 1: GND -> /USB_TXN
- C30 pad 2: Net-(C30-Pad2) -> /FT_TODN
- C31 pad 1: Net-(C31-Pad1) -> /USB_TXP
- C31 pad 2: GND -> /FT_TODP
- C33 pad 1: +3V3 -> GND
- C33 pad 2: GND -> Net-(C33-Pad2)
- C34 pad 1: VD10 -> GND
- C34 pad 2: GND -> Net-(C34-Pad2)
- C35 pad 1: VD10 -> +3V3
- C37 pad 1: +3V3 -> VD10
- C6 pad 1: Net-(C6-Pad1) -> +5V
- D1 pad 1: GND -> Net-(D1-Pad1)
- D1 pad 2: Net-(D1-Pad2) -> +3V3
- FB1 pad 2: +5V -> VBUS
- J4 pad 1: GND -> Net-(J4-Pad1)
- J4 pad 2: /JTAG_TDI -> Net-(J4-Pad2)
- J4 pad 3: /JTAG_TMS -> Net-(J4-Pad3)
- J4 pad 4: /JTAG_TDO -> Net-(J4-Pad4)
- J4 pad 5: /JTAG_TCK -> Net-(J4-Pad5)
- J4 pad 6: +3V3 -> Net-(J4-Pad6)
- J5 pad 1: /USB_DP -> /PMOD0_0
- J5 pad 10: Net-(J5-Pad10) -> /PMOD0_5
- J5 pad 2: /USB_DM -> /PMOD0_1
- J5 pad 3: GND -> /PMOD0_2
- J5 pad 4: /FT_RIDN -> /PMOD0_3
- J5 pad 5: /FT_RIDP -> GND
- J5 pad 6: /FT_TODP -> /PMOD0_VCC
- J5 pad 7: /FT_TODN -> /PMOD0_VCC
- J5 pad 9: Net-(J5-Pad9) -> /PMOD0_4
- L1 pad 1: Net-(C13-Pad2) -> Net-(C14-Pad2)
- L1 pad 2: Net-(C19-Pad1) -> Net-(C20-Pad1)
- L2 pad 1: Net-(C14-Pad2) -> Net-(C15-Pad2)
- L2 pad 2: Net-(C20-Pad1) -> Net-(C21-Pad1)
- L3 pad 1: Net-(C15-Pad2) -> Net-(C16-Pad2)
- L3 pad 2: Net-(C21-Pad1) -> Net-(C22-Pad1)
- R1 pad 1: Net-(R1-Pad1) -> +3V3
- R1 pad 2: GND -> Net-(R1-Pad2)
- R10 pad 1: Net-(C20-Pad1) -> Net-(C20-Pad2)
- R10 pad 2: Net-(C20-Pad2) -> GND
- R11 pad 1: Net-(C20-Pad2) -> Net-(C21-Pad1)
- R11 pad 2: GND -> Net-(C21-Pad2)
- R12 pad 1: Net-(C21-Pad1) -> Net-(C21-Pad2)
- R12 pad 2: Net-(C21-Pad2) -> GND
- R13 pad 1: Net-(C21-Pad2) -> Net-(C22-Pad1)
- R13 pad 2: GND -> Net-(C22-Pad2)
- R14 pad 1: +2V5 -> Net-(C22-Pad2)
- R14 pad 2: Net-(C20-Pad1) -> GND
- R15 pad 1: +3V3 -> /PROGRAMn
- R15 pad 2: Net-(C21-Pad1) -> FT_GPIO0
- R16 pad 1: +1V8 -> Net-(D2-Pad1)
- R16 pad 2: Net-(C6-Pad1) -> GND
- R17 pad 1: +1V1 -> +2V5
- R17 pad 2: Net-(C19-Pad1) -> Net-(C21-Pad1)
- R18 pad 1: GND -> +3V3
- R18 pad 2: Net-(J3-PadA5) -> Net-(C22-Pad1)
- R19 pad 1: GND -> +1V8
- R19 pad 2: Net-(J3-PadB5) -> Net-(C7-Pad1)
- R2 pad 2: Net-(D1-Pad2) -> GND
- R20 pad 1: /FT_DM -> /PROGRAMn
- R20 pad 2: /USB_DM -> +3V3
- R21 pad 1: /FT_DP -> +1V1
- R21 pad 2: /USB_DP -> Net-(C20-Pad1)
- R22 pad 1: Net-(R22-Pad1) -> /INITn
- R22 pad 2: Net-(J3-PadA8) -> +3V3
- R23 pad 1: Net-(R23-Pad1) -> Net-(C28-Pad1)
- R23 pad 2: Net-(J3-PadB8) -> GND
- R24 pad 1: Net-(R24-Pad1) -> Net-(C29-Pad1)
- R25 pad 1: Net-(R25-Pad1) -> GND
- R25 pad 2: +3V3 -> Net-(J2-PadA5)
- R26 pad 1: Net-(R26-Pad1) -> GND
- R26 pad 2: +3V3 -> Net-(J2-PadB5)
- R27 pad 1: Net-(R27-Pad1) -> /FT_DM
- R27 pad 2: +3V3 -> /USB_DM
- R28 pad 1: /FT_BE_0 -> /FT_DP
- R28 pad 2: Net-(R28-Pad2) -> /USB_DP
- R29 pad 1: /FT_BE_1 -> Net-(R29-Pad1)
- R29 pad 2: Net-(R29-Pad2) -> Net-(J2-PadA8)
- R3 pad 1: +3V3 -> GND
- R30 pad 1: /FT_TXE_N -> Net-(R30-Pad1)
- R30 pad 2: Net-(R30-Pad2) -> Net-(J2-PadB8)
- R31 pad 1: /FT_RXF_N -> Net-(R31-Pad1)
- R31 pad 2: Net-(R31-Pad2) -> GND
- R32 pad 1: /FT_WR_N -> Net-(R32-Pad1)
- R32 pad 2: Net-(R32-Pad2) -> +3V3
- R33 pad 1: /FT_RD_N -> Net-(R33-Pad1)
- R33 pad 2: Net-(R33-Pad2) -> +3V3
- R34 pad 1: /FT_OE_N -> Net-(R34-Pad1)
- R34 pad 2: Net-(R34-Pad2) -> +3V3
- R35 pad 1: /FT_CLK -> /FT_BE_0
- R36 pad 1: /FT_DATA_0 -> /FT_BE_1
- R37 pad 1: /FT_DATA_1 -> /FT_TXE_N
- R38 pad 1: /FT_DATA_2 -> /FT_RXF_N
- R39 pad 1: /FT_DATA_3 -> /FT_WR_N
- R4 pad 1: GND -> /JTAG_TCK
- R4 pad 2: Net-(R4-Pad2) -> GND
- R40 pad 1: /FT_DATA_4 -> /FT_RD_N
- R41 pad 1: /FT_DATA_5 -> /FT_OE_N
- R42 pad 1: /FT_DATA_6 -> /FT_CLK
- R43 pad 1: /FT_DATA_7 -> /FT_DATA_0
- R44 pad 1: /FT_DATA_8 -> /FT_DATA_1
- R45 pad 1: /FT_DATA_9 -> /FT_DATA_2
- R46 pad 1: /FT_DATA_10 -> /FT_DATA_3
- R47 pad 1: /FT_DATA_11 -> /FT_DATA_4
- R48 pad 1: /FT_DATA_12 -> /FT_DATA_5
- R49 pad 1: /FT_DATA_13 -> /FT_DATA_6
- R5 pad 1: Net-(C10-Pad1) -> Net-(C11-Pad1)
- R5 pad 2: Net-(C16-Pad1) -> Net-(C17-Pad1)
- R50 pad 1: /FT_DATA_14 -> /FT_DATA_7
- R51 pad 1: /FT_DATA_15 -> /FT_DATA_8
- R52 pad 1: Net-(C28-Pad1) -> /FT_DATA_9
- R52 pad 2: GND -> Net-(R52-Pad2)
- R53 pad 1: Net-(C31-Pad1) -> /FT_DATA_10
- R53 pad 2: GND -> Net-(R53-Pad2)
- R54 pad 1: /JTAG_TCK -> /FT_DATA_11
- R54 pad 2: GND -> Net-(R54-Pad2)
- R6 pad 1: Net-(C11-Pad1) -> Net-(C12-Pad1)
- R6 pad 2: Net-(C17-Pad1) -> Net-(C18-Pad1)
- R7 pad 1: Net-(C12-Pad1) -> Net-(C13-Pad1)
- R7 pad 2: Net-(C18-Pad1) -> Net-(C19-Pad1)
- R8 pad 1: Net-(C19-Pad1) -> Net-(D1-Pad1)
- R8 pad 2: Net-(C19-Pad2) -> GND
- R9 pad 1: Net-(C19-Pad2) -> Net-(C20-Pad1)
- R9 pad 2: GND -> Net-(C20-Pad2)
- TP1 pad 1: +2V5 -> /PROGRAMn
- TP2 pad 1: +3V3 -> +2V5
- TP3 pad 1: +1V8 -> +3V3
- TP4 pad 1: +1V1 -> +1V8
- U1 pad 1: Net-(U1-Pad1) -> +3V3
- U1 pad 2: Net-(U1-Pad2) -> GND
- U1 pad 3: Net-(U1-Pad3) -> CLK_16MHz
- U1 pad 4: Net-(C1-Pad1) -> +3V3
- U4 pad 1: VD10 -> +5V
- U4 pad 2: Net-(R28-Pad2) -> GND
- U4 pad 3: Net-(R29-Pad2) -> +5V
- U4 pad 4: Net-(R30-Pad2) -> Net-(U4-Pad4)
- U4 pad 5: Net-(R31-Pad2) -> Net-(C7-Pad1)
- U6 pad 1: +3V3 -> VD10
- U6 pad 2: GND -> Net-(R35-Pad2)
- U6 pad 3: CLK_16MHz -> Net-(R36-Pad2)
- U6 pad 4: +3V3 -> Net-(R37-Pad2)
- Y1 pad 1: Net-(C29-Pad2) -> Net-(C33-Pad2)
- Y1 pad 3: Net-(C30-Pad2) -> Net-(C34-Pad2)
Routing:
- net /FT_RIDN: track 0.00 -> 34.5 mm, vias 0 -> 3
- net /FT_RIDP: track 0.00 -> 34.1 mm, vias 0 -> 4
- net /USB_TXP: track 0.00 -> 21.4 mm, vias 0 -> 3
- net /USB_TXN: track 0.00 -> 20.8 mm, vias 0 -> 3
- net VBUS: track 0.00 -> 20.2 mm, vias 0 -> 3
- net GND: track 0.00 -> 18.4 mm, vias 0 -> 6
- net /USB_DM: track 0.00 -> 14.1 mm, vias 0 -> 2
- net /USB_DP: track 0.00 -> 13.8 mm, vias 0 -> 2
- net Net-(J2-PadB5): track 0.00 -> 11.3 mm, vias 0 -> 2
- net Net-(J2-PadA5): track 0.00 -> 9.32 mm, vias 0 -> 2
- net Net-(J2-PadB8): track 0.00 -> 8.18 mm, vias 0 -> 2
- net /FT_TODN: track 0.00 -> 3.49 mm
- net /FT_DM: track 0.00 -> 3.46 mm
- net /FT_TODP: track 0.00 -> 3.08 mm
- net /FT_DP: track 0.00 -> 3.05 mm
- added copper zone on In2.Cu, net +3V3
- added copper zone on In1.Cu, net GND
- added copper zone on In2.Cu, net VBUS
- removed copper zone on F.Cu, net GND
Other:
- board size 95 x 95 mm -> 95 x 80 mm
- copper layers 2 -> 4
- net class Default: clearance 0.2 -> 0.127; trace_width 0.25 -> 0.127; via_dia 0.8 -> 0.45; via_drill 0.4 -> 0.2
- rule trace_clearance: 0.2 -> 0.127
- rule trace_min: 0.2 -> 0.127
- rule via_min_drill: 0.3 -> 0.2
- rule via_min_size: 0.4 -> 0.45

Commit message: asdf
Routing:
- net /FT_TODN: track 3.49 -> 10.5 mm, vias 0 -> 2
- net /FT_DM: track 3.46 -> 9.75 mm
- net /FT_DP: track 3.05 -> 9.21 mm
- net /FT_TODP: track 3.08 -> 9.20 mm
- net +3V3: track 0.00 -> 2.82 mm, vias 0 -> 1
Changed lines of the file:
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@@
     (thickness 1.6)
     (drawings 8)
-    (tracks 223)
+    (tracks 250)
     (zones 0)
     (modules 158)
@@
   (segment (start 60.4 94.75) (end 60.4 94.9) (width 0.3) (layer F.Cu) (net 1))
   (segment (start 58.515 92.865) (end 60.4 94.75) (width 0.3) (layer F.Cu) (net 1))
+  (segment (start 71.524999 88.924999) (end 71.3 88.7) (width 0.127) (layer F.Cu) (net 2))
+  (segment (start 71.6 89) (end 71.524999 88.924999) (width 0.127) (layer F.Cu) (net 2))
+  (segment (start 74 89) (end 71.6 89) (width 0.127) (layer F.Cu) (net 2))
+  (via (at 71.3 88.7) (size 0.45) (drill 0.2) (layers F.Cu B.Cu) (net 2))
   (segment (start 67.3125 88) (end 68.0875 88) (width 0.127) (layer F.Cu) (net 186))
   (segment (start 65.0375 88) (end 67.3125 88) (width 0.127) (layer F.Cu) (net 186))
+  (segment (start 68.452 88) (end 68.0875 88) (width 0.127) (layer F.Cu) (net 186))
+  (segment (start 71.3 88) (end 68.452 88) (width 0.127) (layer F.Cu) (net 186))
+  (segment (start 74 88.6) (end 71.9 88.6) (width 0.127) (layer F.Cu) (net 186))
+  (segment (start 71.9 88.6) (end 71.3 88) (width 0.127) (layer F.Cu) (net 186))
   (segment (start 67.3125 88.5) (end 68.0875 88.5) (width 0.127) (layer F.Cu) (net 187))
   (segment (start 66.575 88.5) (end 67.3125 88.5) (width 0.127) (layer F.Cu) (net 187))
   (segment (start 65.0375 89.5) (end 65.575 89.5) (width 0.127) (layer F.Cu) (net 187))
   (segment (start 65.575 89.5) (end 66.575 88.5) (width 0.127) (layer F.Cu) (net 187))
+  (segment (start 68.452 88.5) (end 68.0875 88.5) (width 0.127) (layer F.Cu) (net 187))
+  (segment (start 70.181277 89.290501) (end 69.390776 88.5) (width 0.127) (layer F.Cu) (net 187))
+  (segment (start 69.390776 88.5) (end 68.452 88.5) (width 0.127) (layer F.Cu) (net 187))
+  (segment (start 74 89.4) (end 73.890501 89.290501) (width 0.127) (layer F.Cu) (net 187))
+  (segment (start 73.890501 89.290501) (end 70.181277 89.290501) (width 0.127) (layer F.Cu) (net 187))
   (segment (start 67.302434 91.412249) (end 68.077434 91.412249) (width 0.127) (layer F.Cu) (net 189))
   (segment (start 66.587751 91.412249) (end 67.302434 91.412249) (width 0.127) (layer F.Cu) (net 189))
@@
   (segment (start 65.0375 92.5) (end 65.2 92.5) (width 0.127) (layer F.Cu) (net 189))
   (segment (start 65.2 92.5) (end 66.287751 91.412249) (width 0.127) (layer F.Cu) (net 189))
+  (via (at 71.75 91.327749) (size 0.45) (drill 0.2) (layers F.Cu B.Cu) (net 189))
+  (segment (start 69.057309 91.327749) (end 71.75 91.327749) (width 0.127) (layer F.Cu) (net 189))
+  (segment (start 68.077434 91.412249) (end 68.972809 91.412249) (width 0.127) (layer F.Cu) (net 189))
+  (segment (start 68.972809 91.412249) (end 69.057309 91.327749) (width 0.127) (layer F.Cu) (net 189))
+  (via (at 71.75 90.496749) (size 0.45) (drill 0.2) (layers F.Cu B.Cu) (net 189))
+  (segment (start 71.75 91.327749) (end 71.75 90.496749) (width 0.127) (layer B.Cu) (net 189))
+  (segment (start 73.473 91) (end 74 91) (width 0.127) (layer F.Cu) (net 189))
+  (segment (start 72.5 91) (end 73.473 91) (width 0.127) (layer F.Cu) (net 189))
+  (segment (start 71.75 90.496749) (end 71.996749 90.496749) (width 0.127) (layer F.Cu) (net 189))
+  (segment (start 71.996749 90.496749) (end 72.5 91) (width 0.127) (layer F.Cu) (net 189))
   (segment (start 67.302434 90.912249) (end 68.077434 90.912249) (width 0.127) (layer F.Cu) (net 192))
   (segment (start 66.787751 90.912249) (end 67.302434 90.912249) (width 0.127) (layer F.Cu) (net 192))
   (segment (start 65.0375 91) (end 66.7 91) (width 0.127) (layer F.Cu) (net 192))
   (segment (start 66.7 91) (end 66.787751 90.912249) (width 0.127) (layer F.Cu) (net 192))
+  (segment (start 72.540776 91.4) (end 72.053025 90.912249) (width 0.127) (layer F.Cu) (net 192))
+  (segment (start 74 91.4) (end 72.540776 91.4) (width 0.127) (layer F.Cu) (net 192))
+  (segment (start 68.441934 90.912249) (end 68.077434 90.912249) (width 0.127) (layer F.Cu) (net 192))
+  (segment (start 72.053025 90.912249) (end 68.441934 90.912249) (width 0.127) (layer F.Cu) (net 192))
   (segment (start 67.302434 92.912249) (end 68.077434 92.912249) (width 0.127) (layer F.Cu) (net 193))
   (via (at 60.299992 93.4) (size 0.45) (drill 0.2) (layers F.Cu B.Cu) (net 193))

Commit message: Routing
Parts:
- removed C28, C29: 100n, Capacitor_SMD:C_0603_1608Metric
- removed R23, R24: 1M, Resistor_SMD:R_0603_1608Metric
- removed R26: 5K1, Resistor_SMD:R_0603_1608Metric
- removed R30: 0R, Resistor_SMD:R_0603_1608Metric
- moved U3 94.4 mm to (66.5, 69.0)
- moved FB1 65.2 mm to (55.0, 81.0), turned to 270 degrees
- moved R31 42.5 mm to (66.7, 96.5)
- moved J3 29.5 mm to (53.2, 102.5)
- moved R29 17.0 mm to (60.0, 97.0), turned to 90 degrees
- moved R25 12.8 mm to (64.5, 93.8), turned to 180 degrees
- moved J7 4.48 mm to (65.9, 87.8)
- moved C30 4.37 mm to (62.5, 88.5)
- moved C31 4.37 mm to (62.5, 87.0)
- moved U6 4.00 mm to (73.5, 90.0)
- moved J6 2.69 mm to (65.9, 91.0), turned to 270 degrees
- moved R27 2.66 mm to (62.5, 91.5)
- moved R28 2.66 mm to (62.5, 90.0)
Connections:
- J2 pad A10: /FT_RIDN -> Net-(J2-PadA10)
- J2 pad A11: /FT_RIDP -> Net-(J2-PadA11)
- J2 pad B2: /USB_TXP -> Net-(J2-PadB2)
- J2 pad B3: /USB_TXN -> Net-(J2-PadB3)
- J2 pad B6: /USB_DP -> Net-(J2-PadB6)
- J2 pad B7: /USB_DM -> Net-(J2-PadB7)
- J3 pad 6: Net-(C29-Pad1) -> GND
- J6 pad 1: Net-(J6-Pad1) -> /FT_DP
- J6 pad 10: Net-(J6-Pad10) -> /FT_DP
- J6 pad 2: Net-(J6-Pad2) -> /FT_DM
- J6 pad 4: /FT_DM -> Net-(J6-Pad4)
- J6 pad 5: /FT_DP -> Net-(J6-Pad5)
- J6 pad 6: /FT_DP -> Net-(J6-Pad6)
- J6 pad 7: /FT_DM -> Net-(J6-Pad7)
- J6 pad 9: Net-(J6-Pad9) -> /FT_DM
Routing:
- net GND: track 18.4 -> 36.3 mm, vias 6 -> 9
- net /USB_TXP: track 21.4 -> 3.81 mm, vias 3 -> 0
- net /USB_TXN: track 20.8 -> 3.63 mm, vias 3 -> 0
- net /FT_RIDN: track 34.5 -> 18.8 mm, vias 3 -> 4
- net /FT_RIDP: track 34.1 -> 19.4 mm
- net Net-(J2-PadB5): track 11.3 -> 0.00 mm, vias 2 -> 0
- net Net-(J2-PadB8): track 8.18 -> 0.00 mm, vias 2 -> 0
- net Net-(J2-PadA8): track 0.00 -> 7.78 mm
- net /USB_DP: track 13.8 -> 21.5 mm, vias 2 -> 0
- net VBUS: track 20.2 -> 12.9 mm, vias 3 -> 5
- net /USB_DM: track 14.1 -> 19.2 mm, vias 2 -> 0
- net +3V3: track 2.82 -> 7.31 mm, vias 1 -> 5
- net Net-(J2-PadA5): track 9.32 -> 4.86 mm
- net /FT_TODP: track 9.20 -> 11.4 mm, vias 0 -> 2
- net /FT_DM: track 9.75 -> 7.61 mm
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Other:
- net class Power added: clearance 0.127, trace_width 0.28, via_dia 0.8, via_drill 0.4

Commit message: yarrr. fixed imoprtant pmic bug
Parts:
- J3: footprint Connector_USB:USB_Micro-B_Molex_47346-0001 -> Connector_USB:USB_Micro-B_Molex-105017-0001
- L1, L2, L3: footprint Inductor_SMD:L_0603_1608Metric -> L_1008_1210:L_1008_1210
- moved R35 153.0 mm to (194.7, 88.9)
- moved R36 153.0 mm to (193.7, 92.9)
- moved R37 153.0 mm to (192.7, 88.9)
- moved R38 153.0 mm to (191.7, 92.9)
- moved R39 153.0 mm to (190.7, 88.9)
- moved R40 153.0 mm to (189.7, 92.9)
- moved R41 153.0 mm to (188.7, 88.9)
- moved R42 153.0 mm to (187.7, 92.9)
- moved R43 153.0 mm to (186.7, 88.9)
- moved R44 153.0 mm to (185.7, 92.9)
- moved R45 153.0 mm to (184.7, 88.9)
- moved R46 153.0 mm to (183.7, 92.9)
- moved R47 153.0 mm to (182.7, 88.9)
- moved R48 153.0 mm to (181.7, 92.9)
- moved R49 153.0 mm to (180.7, 88.9)
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Connections:
- U3 pad 10: Net-(C15-Pad1) -> Net-(C15-Pad2)
- U3 pad 15: Net-(C16-Pad1) -> Net-(C16-Pad2)
- U3 pad 16: Net-(C16-Pad2) -> Net-(C16-Pad1)
- U3 pad 9: Net-(C15-Pad2) -> Net-(C15-Pad1)
Routing:
- net GND: track 36.3 -> 112.3 mm, vias 9 -> 111
- net +1V1: track 0.00 -> 25.7 mm, vias 0 -> 6
- net Net-(C33-Pad2): track 0.00 -> 7.63 mm
- net Net-(C34-Pad2): track 0.00 -> 6.46 mm
- net +5V: track 0.00 -> 6.18 mm, vias 0 -> 3
- net Net-(C15-Pad1): track 0.00 -> 5.12 mm
- net +3V3: track 7.31 -> 11.8 mm, vias 5 -> 13
- net Net-(C15-Pad2): track 0.00 -> 2.44 mm
- added copper zone on B.Cu, net +1V1
- added copper zone on B.Cu, net GND
- added copper zone on F.Cu, net GND
- added copper zone on F.Cu, net Net-(C15-Pad2)
- added copper zone on F.Cu, net Net-(C16-Pad2)
Other:
- net class Default: clearance 0.127 -> 0.1016
- net class TightAsFuck added: clearance 0.0889, trace_width 0.0889, via_dia 0.45, via_drill 0.2
- rule trace_clearance: 0.127 -> 0.1016
- rule trace_min: 0.127 -> 0.0889
