File: Kilsyth.kicad_pcb (KiCad board)
At the start: 4 copper layers, 95 x 80 mm, 152 parts, among them J1 Conn_JTAG, J2 DX07S024JJ2, J3 USB_B_Micro, J4 Conn_02x20_Counter_Clockwise, J5 Conn_02x06_Counter_Clockwise, J6 PUSB3FR4Z, J7 PUSB3FR4Z, J8 Conn_02x06_Counter_Clockwise, J9 Conn_02x06_Counter_Clockwise, SW1 SW_Push, U1 DSC6001CI2A-016.0000T, U2 LFE5U-85F-6BG381C, U3 TPS65261, U4 MIC5504-1.8YM5, U5 IS25LP128F-JBLE, U6 FT600Q, U7 AS4C32M16SB, Y1 30MHz ±20ppm

Commit message: Some progress
Parts:
- moved R14 108.5 mm to (71.8, 55.2), turned to 90 degrees
- moved R13 104.4 mm to (68.8, 55.2), turned to 270 degrees
- moved C22 104.4 mm to (70.3, 55.2), turned to 270 degrees
- moved R18 102.8 mm to (78.7, 62.4), turned to 270 degrees
- moved C14 102.6 mm to (63.3, 62.0), turned to 180 degrees
- moved C13 102.3 mm to (71.6, 59.0)
- moved C20 101.4 mm to (62.8, 55.2), turned to 270 degrees
- moved C10 99.4 mm to (71.6, 60.5)
- moved R21 98.4 mm to (54.1, 62.7), turned to 270 degrees
- moved C19 97.7 mm to (73.3, 55.2), turned to 90 degrees
- moved C3 91.2 mm to (75.5, 69.5), turned to 270 degrees
- moved R11 90.5 mm to (71.9, 78.0), turned to 180 degrees
- moved R10 87.3 mm to (65.8, 55.2), turned to 90 degrees
- moved C21 85.5 mm to (71.9, 76.5), turned to 180 degrees
- moved C45 84.2 mm to (86.1, 77.6)
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Routing:
- net GND: track 112.3 -> 137.3 mm, vias 111 -> 134
- net +2V5: track 0.00 -> 24.2 mm, vias 0 -> 16
- net Net-(C22-Pad1): track 0.00 -> 19.1 mm, vias 0 -> 2
- net Net-(C20-Pad1): track 0.00 -> 13.8 mm
- net Net-(C20-Pad2): track 0.00 -> 13.6 mm
- net Net-(C22-Pad2): track 0.00 -> 13.2 mm
- net Net-(C21-Pad2): track 0.00 -> 11.7 mm, vias 0 -> 2
- net Net-(R2-Pad1): track 0.00 -> 10.3 mm
- net Net-(C11-Pad1): track 0.00 -> 9.52 mm
- net Net-(C13-Pad1): track 0.00 -> 9.28 mm
- net Net-(C2-Pad1): track 0.00 -> 7.82 mm
- net +3V3: track 11.8 -> 18.6 mm, vias 13 -> 37
- net Net-(C21-Pad1): track 0.00 -> 6.72 mm
- net +5V: track 6.18 -> 12.5 mm, vias 3 -> 8
- net Net-(C8-Pad1): track 0.00 -> 6.31 mm
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- added copper zone on F.Cu, net +1V1
- added copper zone on In2.Cu, net +1V1
- added copper zone on F.Cu, net +2V5
- added copper zone on F.Cu, net +3V3
- added copper zone on B.Cu, net +5V
- added copper zone on F.Cu, net +5V
- added copper zone on F.Cu, net Net-(C14-Pad2)
- added copper zone on F.Cu, net Net-(C20-Pad1)
- added copper zone on F.Cu, net Net-(C21-Pad1)
- added copper zone on F.Cu, net Net-(C22-Pad1)
- added copper zone on F.Cu, net VBUS

Commit message: woop
Parts:
- moved R35 145.7 mm to (63.6, 152.5)
- moved R36 145.7 mm to (62.6, 156.5)
- moved R37 145.7 mm to (61.6, 152.5)
- moved R38 145.7 mm to (60.6, 156.5)
- moved R39 145.7 mm to (59.6, 152.5)
- moved R40 145.7 mm to (58.6, 156.5)
- moved R41 145.7 mm to (57.6, 152.5)
- moved R42 145.7 mm to (56.6, 156.5)
- moved R43 145.7 mm to (55.6, 152.5)
- moved R44 145.7 mm to (54.6, 156.5)
- moved R45 145.7 mm to (53.6, 152.5)
- moved R46 145.7 mm to (52.6, 156.5)
- moved R47 145.7 mm to (51.6, 152.5)
- moved R48 145.7 mm to (50.6, 156.5)
- moved R49 145.7 mm to (49.6, 152.5)
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Connections:
- U2 pad A2: /RAM_DQ7 -> /BANK7
- U2 pad A3: /RAM_DQ0 -> /BANK7
- U2 pad A4: Net-(U2-PadA4) -> /BANK7
- U2 pad A5: /RAM_A0 -> /BANK7
- U2 pad B1: /RAM_A8 -> /BANK7
- U2 pad B2: /RAM_DQ6 -> /BANK7
- U2 pad B3: /RAM_A1 -> /BANK7
- U2 pad B4: /RAM_A2 -> /BANK7
- U2 pad B5: Net-(U2-PadB5) -> /BANK7
- U2 pad C1: /RAM_DQ9 -> /BANK7
- U2 pad C18: /BANK2 -> Net-(U2-PadC18)
- U2 pad C2: /RAM_A7 -> /BANK7
- U2 pad C20: /BANK2 -> /RAM_DQ9
- U2 pad C3: /RAM_DQ2 -> /BANK7
- U2 pad C4: /RAM_DQ1 -> /BANK7
- U2 pad C5: Net-(U2-PadC5) -> /BANK7
- U2 pad D1: /RAM_A10 -> /BANK7
- U2 pad D17: /BANK2 -> Net-(U2-PadD17)
- U2 pad D18: /BANK2 -> Net-(U2-PadD18)
- U2 pad D19: /BANK2 -> /RAM_DQ10
- U2 pad D2: /RAM_DQ8 -> /BANK7
- U2 pad D20: /BANK2 -> /RAM_DQ11
- U2 pad D3: /RAM_A3 -> /BANK7
- U2 pad D5: /RAM_A4 -> /BANK7
- U2 pad E1: /RAM_A9 -> /BANK7
- U2 pad E16: /BANK2 -> Net-(U2-PadE16)
- U2 pad E17: /BANK2 -> Net-(U2-PadE17)
- U2 pad E18: /BANK2 -> /RAM_DQ12
- U2 pad E19: /BANK2 -> /RAM_DQ8
- U2 pad E2: /RAM_DQ15 -> /BANK7
- U2 pad E20: /BANK2 -> /RAM_DQM1
- U2 pad E3: /RAM_A6 -> /BANK7
- U2 pad E4: /RAM_DQ3 -> /BANK7
- U2 pad E5: /RAM_DQ4 -> /BANK7
- U2 pad F1: /RAM_DQM1 -> /BANK6
- U2 pad F16: /BANK2 -> Net-(U2-PadF16)
- U2 pad F17: /BANK2 -> Net-(U2-PadF17)
- U2 pad F18: /BANK2 -> /RAM_DQ13
- U2 pad F19: /BANK2 -> /RAM_CLK
- U2 pad F2: /RAM_DQ12 -> /BANK7
- U2 pad F20: /BANK2 -> /RAM_CKE
- U2 pad F3: /RAM_DQ14 -> /BANK7
- U2 pad F4: /RAM_DQ5 -> /BANK7
- U2 pad F5: /RAM_A5 -> /BANK7
- U2 pad G1: /RAM_DQM0 -> /BANK6
- U2 pad G16: /BANK2 -> Net-(U2-PadG16)
- U2 pad G18: /BANK2 -> Net-(U2-PadG18)
- U2 pad G19: /BANK2 -> /RAM_A12
- U2 pad G20: /BANK2 -> /RAM_A11
- U2 pad G3: /RAM_DQ13 -> /BANK7
- U2 pad G5: /RAM_A12 -> /BANK7
- U2 pad H16: /BANK2 -> Net-(U2-PadH16)
- U2 pad H17: /BANK2 -> Net-(U2-PadH17)
- U2 pad H18: /BANK2 -> Net-(U2-PadH18)
- U2 pad H20: /BANK2 -> /RAM_A9
- U2 pad H3: /RAM_A11 -> /BANK7
- U2 pad H4: /RAM_DQ11 -> /BANK7
- U2 pad H5: /RAM_DQ10 -> /BANK7
- U2 pad J1: Net-(U2-PadJ1) -> /BANK6
- U2 pad J16: /BANK2 -> Net-(U2-PadJ16)
- U2 pad J17: /BANK2 -> /RAM_DQ15
- U2 pad J18: /BANK2 -> /RAM_DQ14
- U2 pad J19: /BANK2 -> /RAM_A8
- U2 pad J20: /BANK2 -> /RAM_A7
- U2 pad J5: Net-(U2-PadJ5) -> /BANK6
- U2 pad K1: Net-(U2-PadK1) -> /BANK6
- U2 pad K18: /BANK2 -> /RAM_A6
- U2 pad K19: /BANK2 -> /RAM_A5
- U2 pad K20: /BANK2 -> /RAM_A4
- U2 pad K3: Net-(U2-PadK3) -> /BANK6
- U2 pad K5: /RAM_BA0 -> /BANK6
- U2 pad L16: /BANK3 -> Net-(U2-PadL16)
- U2 pad L17: /BANK3 -> Net-(U2-PadL17)
- U2 pad L18: /BANK3 -> Net-(U2-PadL18)
- U2 pad L19: /BANK3 -> /RAM_A3
- U2 pad L2: /RAM_~RAS -> /BANK6
- U2 pad L20: /BANK3 -> /RAM_A2
- U2 pad L5: Net-(U2-PadL5) -> /BANK6
- U2 pad M1: /RAM_CLK -> /BANK6
- U2 pad M17: /BANK3 -> Net-(U2-PadM17)
- U2 pad M18: /BANK3 -> Net-(U2-PadM18)
- U2 pad M19: /BANK3 -> /RAM_A1
- U2 pad M20: /BANK3 -> /RAM_A0
- U2 pad M3: /RAM_~CAS -> /BANK6
- U2 pad N1: /RAM_~WE -> /BANK6
- U2 pad N16: /BANK3 -> Net-(U2-PadN16)
- U2 pad N17: /BANK3 -> Net-(U2-PadN17)
- U2 pad N18: /BANK3 -> /RAM_DQ3
- U2 pad N19: /BANK3 -> /RAM_A10
- U2 pad N20: /BANK3 -> /RAM_BA1
- U2 pad N5: /RAM_~CS -> /BANK6
- U2 pad P16: /BANK3 -> Net-(U2-PadP16)
- U2 pad P17: /BANK3 -> Net-(U2-PadP17)
- U2 pad P18: /BANK3 -> Net-(U2-PadP18)
- U2 pad P19: /BANK3 -> /RAM_BA0
- U2 pad P2: Net-(U2-PadP2) -> /BANK6
- U2 pad P20: /BANK3 -> /RAM_~CS
- U2 pad P4: /RAM_CKE -> /BANK6
- U2 pad P5: /RAM_BA1 -> /BANK6
- U2 pad R16: /BANK3 -> Net-(U2-PadR16)
- U2 pad R17: /BANK3 -> /RAM_DQ4
- U2 pad R18: /BANK3 -> Net-(U2-PadR18)
- U2 pad R20: /BANK3 -> /RAM_~RAS
- U2 pad T17: /BANK3 -> /RAM_DQ6
- U2 pad T18: /BANK3 -> /RAM_DQ5
- U2 pad T19: /BANK3 -> /RAM_~CAS
- U2 pad T20: /BANK3 -> /RAM_~WE
- U2 pad U16: /BANK3 -> /RAM_DQ2
- U2 pad U17: /BANK3 -> /RAM_DQ1
- U2 pad U18: /BANK3 -> /RAM_DQ0
- U2 pad U19: /BANK3 -> /RAM_DQM0
- U2 pad U20: /BANK3 -> /RAM_DQ7
Routing:
- net /RAM_A3: track 0.00 -> 34.6 mm
- net /RAM_A5: track 0.00 -> 34.1 mm
- net /RAM_A4: track 0.00 -> 33.9 mm
- net /RAM_A6: track 0.00 -> 33.9 mm, vias 0 -> 2
- net /RAM_A1: track 0.00 -> 32.7 mm
- net /RAM_A2: track 0.00 -> 32.7 mm
- net /RAM_A8: track 0.00 -> 31.2 mm
- net /RAM_A10: track 0.00 -> 31.1 mm
- net /RAM_A7: track 0.00 -> 31.0 mm
- net /RAM_A0: track 0.00 -> 30.9 mm
- net /RAM_BA0: track 0.00 -> 29.4 mm
- net /RAM_A9: track 0.00 -> 29.4 mm
- net /RAM_BA1: track 0.00 -> 29.3 mm
- net /RAM_A12: track 0.00 -> 28.8 mm
- net /RAM_A11: track 0.00 -> 28.7 mm
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Other:
- board text added: "+1V1"
- board text added: "+2V2"
- board text added: "+3V3"
