File: Kilsyth.kicad_pcb (KiCad board)
At the start: 4 copper layers, 95 x 80 mm, 152 parts, among them J1 Conn_JTAG, J2 DX07S024JJ2, J3 USB_B_Micro, J4 Conn_02x20_Counter_Clockwise, J5 Conn_02x06_Counter_Clockwise, J6 PUSB3FR4Z, J7 PUSB3FR4Z, J8 Conn_02x06_Counter_Clockwise, J9 Conn_02x06_Counter_Clockwise, SW1 SW_Push, U1 DSC6001CI2A-016.0000T, U2 LFE5U-85F-6BG381C, U3 TPS65261, U4 MIC5504-1.8YM5, U5 IS25LP128F-JBLE, U6 FT600Q, U7 AS4C32M16SB, Y1 30MHz ±20ppm

Commit message: before r0 hell
Parts:
- removed R15: 0R, Resistor_SMD:R_0603_1608Metric
- added R23: 0R, Resistor_SMD:R_0603_1608Metric, F.Cu at (48.0, 146.5)
- added R24: 0R, Resistor_SMD:R_0603_1608Metric, F.Cu at (52.0, 147.5)
- moved R33 86.7 mm to (76.0, 78.8), turned to 90 degrees
- moved R20 84.2 mm to (81.4, 143.8)
- moved R32 63.4 mm to (77.6, 78.8), turned to 90 degrees
- moved R34 62.6 mm to (74.4, 78.8), turned to 90 degrees
- moved TP4 39.5 mm to (44.8, 89.9)
- moved R57 19.0 mm to (48.0, 170.4), turned to 180 degrees
- moved R58 18.8 mm to (52.0, 171.4), turned to 180 degrees
- moved R55 16.5 mm to (48.0, 168.4), turned to 180 degrees
- moved R35 16.1 mm to (48.0, 148.4), turned to 180 degrees
- moved R56 16.0 mm to (52.0, 169.4), turned to 180 degrees
- moved R53 14.1 mm to (48.0, 166.4), turned to 180 degrees
- moved R37 13.8 mm to (48.0, 150.4), turned to 180 degrees
- moved R54 13.2 mm to (52.0, 167.4), turned to 180 degrees
- moved R36 12.7 mm to (52.0, 149.4), turned to 180 degrees
- moved R51 11.9 mm to (48.0, 164.4), turned to 180 degrees
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Connections:
- R20 pad 1: /PROGRAMn -> FT_GPIO0
- SW1 pad 2: /PROGRAMn -> FT_GPIO0
- TP1 pad 1: /PROGRAMn -> FT_GPIO0
- U2 pad A10: /FT_WR_N -> /BANK0
- U2 pad A11: /FT_OE_N -> /BANK0
- U2 pad A6: /FT_DATA_0 -> /BANK0
- U2 pad A7: /FT_DATA_12 -> /BANK0
- U2 pad A8: /FT_DATA_13 -> /BANK0
- U2 pad A9: /FT_RXF_N -> /BANK0
- U2 pad B10: /FT_TXE_N -> /BANK0
- U2 pad B11: /FT_CLK -> /BANK0
- U2 pad B6: /FT_DATA_1 -> /BANK0
- U2 pad B8: /FT_DATA_11 -> /BANK0
- U2 pad B9: /FT_BE_0 -> /BANK0
- U2 pad C10: /FT_DATA_15 -> /BANK0
- U2 pad C11: /FT_RD_N -> /BANK0
- U2 pad C6: /FT_DATA_6 -> /BANK0
- U2 pad C7: /FT_DATA_7 -> /BANK0
- U2 pad C8: /FT_DATA_10 -> /BANK0
- U2 pad C9: Net-(U2-PadC9) -> /BANK0
- U2 pad D10: Net-(U2-PadD10) -> /BANK0
- U2 pad D6: /FT_DATA_3 -> /BANK0
- U2 pad D7: /FT_DATA_5 -> /BANK0
- U2 pad D8: /FT_DATA_9 -> /BANK0
- U2 pad D9: /FT_BE_1 -> /BANK0
- U2 pad E10: Net-(U2-PadE10) -> /BANK0
- U2 pad E6: /FT_DATA_2 -> /BANK0
- U2 pad E7: /FT_DATA_4 -> /BANK0
- U2 pad E8: /FT_DATA_8 -> /BANK0
- U2 pad E9: /FT_DATA_14 -> /BANK0
- U2 pad F1: /BANK6 -> /FT_OE_N
- U2 pad G1: /BANK6 -> /FT_RD_N
- U2 pad G2: /BANK6 -> /FT_WR_N
- U2 pad H1: /BANK6 -> /FT_BE_1
- U2 pad H2: /BANK6 -> /FT_CLK
- U2 pad J1: /BANK6 -> /FT_DATA_13
- U2 pad J3: /BANK6 -> /FT_RXF_N
- U2 pad J4: /BANK6 -> /FT_BE_0
- U2 pad J5: /BANK6 -> /FT_DATA_15
- U2 pad K1: /BANK6 -> /FT_DATA_14
- U2 pad K2: /BANK6 -> /FT_DATA_12
- U2 pad K3: /BANK6 -> /FT_TXE_N
- U2 pad K4: /BANK6 -> /FT_DATA_8
- U2 pad K5: /BANK6 -> /FT_DATA_9
- U2 pad L1: /BANK6 -> Net-(U2-PadL1)
- U2 pad L2: /BANK6 -> /FT_DATA_3
- U2 pad L3: /BANK6 -> /FT_DATA_2
- U2 pad L4: /BANK6 -> /FT_DATA_10
- U2 pad L5: /BANK6 -> /FT_DATA_11
- U2 pad M1: /BANK6 -> Net-(U2-PadM1)
- U2 pad M3: /BANK6 -> /FT_DATA_1
- U2 pad M4: /BANK6 -> /FT_DATA_4
- U2 pad N1: /BANK6 -> Net-(U2-PadN1)
- U2 pad N2: /BANK6 -> Net-(U2-PadN2)
- U2 pad N3: /BANK6 -> /FT_DATA_0
- U2 pad N4: /BANK6 -> /FT_DATA_6
- U2 pad N5: /BANK6 -> /FT_DATA_5
- U2 pad P1: /BANK6 -> Net-(U2-PadP1)
- U2 pad P2: /BANK6 -> Net-(U2-PadP2)
- U2 pad P3: /BANK6 -> Net-(U2-PadP3)
- U2 pad P4: /BANK6 -> Net-(U2-PadP4)
- U2 pad P5: /BANK6 -> /FT_DATA_7
- U2 pad W3: /PROGRAMn -> FT_GPIO0
- U6 pad 12: FT_GPIO0 -> Net-(R23-Pad1)
- U6 pad 13: FT_GPIO1 -> Net-(R24-Pad1)
Routing:
- net +5V: track 12.5 -> 37.0 mm, vias 8 -> 10
- net Net-(R31-Pad1): track 0.00 -> 9.05 mm, vias 0 -> 2
- net Net-(J2-PadA5): track 4.86 -> 13.5 mm
- net Net-(R33-Pad1): track 0.00 -> 8.35 mm, vias 0 -> 2
- net Net-(R32-Pad1): track 0.00 -> 8.35 mm, vias 0 -> 2
- net Net-(R34-Pad1): track 0.00 -> 7.87 mm, vias 0 -> 2
- net GND: track 150.9 -> 158.2 mm, vias 141 -> 152
- net VD10: track 19.5 -> 26.2 mm, vias 1 -> 0
- net +3V3: track 35.3 -> 39.3 mm, vias 43 -> 45

Commit message: ayy
Parts:
- J5, J8, J9: value Conn_02x06_Counter_Clockwise -> Conn_02x06_Odd_Even
- moved R8 103.8 mm to (80.2, 53.1)
- moved R3 98.8 mm to (106.1, 109.5), turned to 180 degrees
- moved R4 87.1 mm to (106.8, 118.6)
- moved D1 85.6 mm to (80.2, 51.5)
- moved R1 81.2 mm to (92.0, 117.4)
- moved R43 77.2 mm to (84.2, 88.2), turned to 180 degrees
- moved R24 77.2 mm to (88.2, 79.3)
- moved R23 77.2 mm to (84.2, 78.3)
- moved R35 77.2 mm to (84.2, 80.2)
- moved R36 77.2 mm to (88.2, 81.2)
- moved R37 77.2 mm to (84.2, 82.2)
- moved R38 77.2 mm to (88.2, 83.2)
- moved R39 77.2 mm to (84.2, 84.2)
- moved R40 77.2 mm to (88.2, 85.2)
- moved R41 77.2 mm to (84.2, 86.2)
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Connections:
- J5 pad 1: /PMOD0_0 -> /PMOD0_1
- J5 pad 10: /PMOD0_5 -> GND
- J5 pad 11: /PMOD0_6 -> /PMOD0_VCC
- J5 pad 12: /PMOD0_7 -> /PMOD0_VCC
- J5 pad 2: /PMOD0_1 -> /PMOD0_2
- J5 pad 3: /PMOD0_2 -> /PMOD0_3
- J5 pad 4: /PMOD0_3 -> /PMOD0_4
- J5 pad 5: GND -> /PMOD0_5
- J5 pad 6: /PMOD0_VCC -> /PMOD0_6
- J5 pad 7: /PMOD0_VCC -> /PMOD0_7
- J5 pad 8: GND -> /PMOD0_8
- J5 pad 9: /PMOD0_4 -> GND
- J8 pad 1: /PMOD1_0 -> /PMOD1_1
- J8 pad 10: /PMOD1_5 -> GND
- J8 pad 11: /PMOD1_6 -> /PMOD1_VCC
- J8 pad 12: /PMOD1_7 -> /PMOD1_VCC
- J8 pad 2: /PMOD1_1 -> /PMOD1_2
- J8 pad 3: /PMOD1_2 -> /PMOD1_3
- J8 pad 4: /PMOD1_3 -> /PMOD1_4
- J8 pad 5: GND -> /PMOD1_5
- J8 pad 6: /PMOD1_VCC -> /PMOD1_6
- J8 pad 7: /PMOD1_VCC -> /PMOD1_7
- J8 pad 8: GND -> /PMOD1_8
- J8 pad 9: /PMOD1_4 -> GND
- J9 pad 1: /PMOD2_0 -> /PMOD2_1
- J9 pad 10: /PMOD2_5 -> GND
- J9 pad 11: /PMOD2_6 -> /PMOD2_VCC
- J9 pad 12: /PMOD2_7 -> /PMOD2_VCC
- J9 pad 2: /PMOD2_1 -> /PMOD2_2
- J9 pad 3: /PMOD2_2 -> /PMOD2_3
- J9 pad 4: /PMOD2_3 -> /PMOD2_4
- J9 pad 5: GND -> /PMOD2_5
- J9 pad 6: /PMOD1_VCC -> /PMOD2_6
- J9 pad 7: /PMOD1_VCC -> /PMOD2_7
- J9 pad 8: GND -> /PMOD2_8
- J9 pad 9: /PMOD2_4 -> GND
- R23 pad 2: FT_GPIO0 -> FT_GPIO1
- R24 pad 2: FT_GPIO1 -> FT_GPIO0
- R35 pad 1: /FT_BE_0 -> /FT_OE_N
- R36 pad 1: /FT_BE_1 -> /FT_RD_N
- R37 pad 1: /FT_TXE_N -> /FT_WR_N
- R39 pad 1: /FT_WR_N -> /FT_TXE_N
- R40 pad 1: /FT_RD_N -> /FT_BE_1
- R41 pad 1: /FT_OE_N -> /FT_BE_0
- R42 pad 1: /FT_CLK -> /FT_DATA_15
- R43 pad 1: /FT_DATA_0 -> /FT_DATA_14
- R44 pad 1: /FT_DATA_1 -> /FT_DATA_13
- R45 pad 1: /FT_DATA_2 -> /FT_DATA_12
- R46 pad 1: /FT_DATA_3 -> /FT_DATA_11
- R47 pad 1: /FT_DATA_4 -> /FT_DATA_10
- R48 pad 1: /FT_DATA_5 -> /FT_DATA_9
- R49 pad 1: /FT_DATA_6 -> /FT_DATA_8
- R50 pad 1: /FT_DATA_7 -> /FT_CLK
- R51 pad 1: /FT_DATA_8 -> /FT_DATA_7
- R52 pad 1: /FT_DATA_9 -> /FT_DATA_6
- R53 pad 1: /FT_DATA_10 -> /FT_DATA_5
- R54 pad 1: /FT_DATA_11 -> /FT_DATA_4
- R55 pad 1: /FT_DATA_12 -> /FT_DATA_3
- R56 pad 1: /FT_DATA_13 -> /FT_DATA_2
- R57 pad 1: /FT_DATA_14 -> /FT_DATA_1
- R58 pad 1: /FT_DATA_15 -> /FT_DATA_0
- U2 pad A19: /PMOD2_0 -> /PMOD2_8
- U2 pad B15: /PMOD0_0 -> /PMOD0_8
- U2 pad E14: /PMOD1_0 -> /PMOD1_8
- U2 pad F1: /FT_OE_N -> Net-(U2-PadF1)
- U2 pad G1: /FT_RD_N -> Net-(U2-PadG1)
- U2 pad G2: /FT_WR_N -> Net-(U2-PadG2)
- U2 pad H1: /FT_BE_1 -> /FT_OE_N
- U2 pad H2: /FT_CLK -> /FT_RD_N
- U2 pad J1: /FT_DATA_13 -> /FT_WR_N
- U2 pad J4: /FT_BE_0 -> /FT_TXE_N
- U2 pad J5: /FT_DATA_15 -> /FT_BE_1
- U2 pad K1: /FT_DATA_14 -> /FT_BE_0
- U2 pad K2: /FT_DATA_12 -> /FT_DATA_15
- U2 pad K3: /FT_TXE_N -> /FT_DATA_14
- U2 pad K4: /FT_DATA_8 -> /FT_DATA_13
- U2 pad K5: /FT_DATA_9 -> Net-(U2-PadK5)
- U2 pad L1: Net-(U2-PadL1) -> /FT_DATA_12
- U2 pad L2: /FT_DATA_3 -> /FT_DATA_11
- U2 pad L3: /FT_DATA_2 -> /FT_DATA_10
- U2 pad L4: /FT_DATA_10 -> Net-(U2-PadL4)
- U2 pad L5: /FT_DATA_11 -> Net-(U2-PadL5)
- U2 pad M1: Net-(U2-PadM1) -> /FT_DATA_9
- U2 pad M3: /FT_DATA_1 -> /FT_DATA_8
- U2 pad M4: /FT_DATA_4 -> /FT_CLK
- U2 pad N1: Net-(U2-PadN1) -> /FT_DATA_7
- U2 pad N2: Net-(U2-PadN2) -> /FT_DATA_6
- U2 pad N3: /FT_DATA_0 -> /FT_DATA_5
- U2 pad N4: /FT_DATA_6 -> /FT_DATA_4
- U2 pad N5: /FT_DATA_5 -> Net-(U2-PadN5)
- U2 pad P1: Net-(U2-PadP1) -> /FT_DATA_3
- U2 pad P2: Net-(U2-PadP2) -> /FT_DATA_2
- U2 pad P3: Net-(U2-PadP3) -> /FT_DATA_1
- U2 pad P4: Net-(U2-PadP4) -> /FT_DATA_0
- U2 pad P5: /FT_DATA_7 -> Net-(U2-PadP5)
- U6 pad 12: Net-(R23-Pad1) -> Net-(R24-Pad1)
- U6 pad 13: Net-(R24-Pad1) -> Net-(R23-Pad1)
- U6 pad 2: Net-(R35-Pad2) -> Net-(R41-Pad2)
- U6 pad 3: Net-(R36-Pad2) -> Net-(R40-Pad2)
- U6 pad 33: Net-(R43-Pad2) -> Net-(R58-Pad2)
- U6 pad 34: Net-(R44-Pad2) -> Net-(R57-Pad2)
- U6 pad 35: Net-(R45-Pad2) -> Net-(R56-Pad2)
- U6 pad 36: Net-(R46-Pad2) -> Net-(R55-Pad2)
- U6 pad 39: Net-(R47-Pad2) -> Net-(R54-Pad2)
- U6 pad 4: Net-(R37-Pad2) -> Net-(R39-Pad2)
- U6 pad 40: Net-(R48-Pad2) -> Net-(R53-Pad2)
- U6 pad 41: Net-(R49-Pad2) -> Net-(R52-Pad2)
- U6 pad 42: Net-(R50-Pad2) -> Net-(R51-Pad2)
- U6 pad 43: Net-(R42-Pad2) -> Net-(R50-Pad2)
- U6 pad 45: Net-(R51-Pad2) -> Net-(R49-Pad2)
- U6 pad 46: Net-(R52-Pad2) -> Net-(R48-Pad2)
- U6 pad 47: Net-(R53-Pad2) -> Net-(R47-Pad2)
- U6 pad 48: Net-(R54-Pad2) -> Net-(R46-Pad2)
- U6 pad 53: Net-(R55-Pad2) -> Net-(R45-Pad2)
- U6 pad 54: Net-(R56-Pad2) -> Net-(R44-Pad2)
- U6 pad 55: Net-(R57-Pad2) -> Net-(R43-Pad2)
- U6 pad 56: Net-(R58-Pad2) -> Net-(R42-Pad2)
- U6 pad 7: Net-(R39-Pad2) -> Net-(R37-Pad2)
- U6 pad 8: Net-(R40-Pad2) -> Net-(R36-Pad2)
- U6 pad 9: Net-(R41-Pad2) -> Net-(R35-Pad2)
Routing:
- net /FLASH_CSn: track 0.00 -> 42.0 mm
- net /FLASH_SCK: track 0.00 -> 41.4 mm, vias 0 -> 2
- net /FLASH_MOSI: track 0.00 -> 40.7 mm, vias 0 -> 2
- net /FLASH_MISO: track 0.00 -> 40.7 mm
- net /FLASH_WPn: track 0.00 -> 37.2 mm
- net /FLASH_HOLDn: track 0.00 -> 36.5 mm, vias 0 -> 2
- net DONE: track 0.00 -> 30.1 mm
- net /JTAG_TCK: track 0.00 -> 27.1 mm, vias 0 -> 2
- net Net-(R3-Pad2): track 0.00 -> 26.3 mm, vias 0 -> 2
- net Net-(R1-Pad2): track 0.00 -> 25.5 mm, vias 0 -> 2
- net /JTAG_TMS: track 0.00 -> 24.9 mm, vias 0 -> 2
- net /JTAG_TDO: track 0.00 -> 23.7 mm
- net /JTAG_TDI: track 0.00 -> 23.0 mm, vias 0 -> 2
- net Net-(R24-Pad1): track 0.00 -> 21.3 mm
- net Net-(R58-Pad2): track 0.00 -> 19.9 mm
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- added copper zone on In2.Cu, net +2V5

Commit message: puh
Parts:
- J1: footprint Connector_PinSocket_2.54mm:PinSocket_2x03_P2.54mm_Vertical_SMD -> Connector_PinHeader_2.54mm:PinHeader_2x03_P2.54mm_Vertical_SMD
- moved U4 83.7 mm to (74.3, 152.0)
- moved D2 79.9 mm to (85.3, 122.1)
- moved R16 70.3 mm to (85.3, 120.5)
- moved R19 60.1 mm to (74.3, 144.3)
- moved C7 56.2 mm to (74.3, 146.0), turned to 180 degrees
Routing:
- net /JTAG_TCK: track 27.1 -> 28.3 mm, vias 2 -> 3
- net +3V3: track 54.2 -> 52.9 mm, vias 47 -> 46
Other:
- board text added: "+2V5"
- board text removed: "+2V2"

Commit message: oy
Connections:
- U2 pad J17: /RAM_DQ15 -> /RAM_DQ14
- U2 pad J18: /RAM_DQ14 -> /RAM_DQ15
- U2 pad N18: /RAM_DQ3 -> Net-(U2-PadN18)
- U2 pad P18: Net-(U2-PadP18) -> /RAM_~RAS
- U2 pad R20: /RAM_~RAS -> /RAM_~CAS
- U2 pad T19: /RAM_~CAS -> /RAM_DQM0
- U2 pad U16: /RAM_DQ2 -> /RAM_DQ3
- U2 pad U18: /RAM_DQ0 -> /RAM_DQ2
- U2 pad U19: /RAM_DQM0 -> /RAM_DQ0
Routing:
- net /RAM_DQ3: track 13.0 -> 22.7 mm, vias 1 -> 2
- net /RAM_DQ2: track 20.1 -> 18.5 mm
- net /RAM_~RAS: track 27.0 -> 28.6 mm
- net /RAM_~CAS: track 27.1 -> 26.0 mm
- net /RAM_DQ15: track 19.5 -> 18.7 mm
- net /RAM_DQ0: track 15.4 -> 14.6 mm
