File: hardware/Kilsyth.sch (KiCad schematic (older format))
At the start: 168 parts, among them J1 Conn_JTAG, J10 Conn_02x01, J11 Conn_02x04_Odd_Even, J12 Conn_02x04_Odd_Even, J2 DX07S024JJ2, J3 USB_B_Micro, J4 Conn_02x20_Odd_Even, J5 Conn_02x06_Odd_Even, J6 PUSB3FR4Z, J7 PUSB3FR4Z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

Commit message: Add errata
Connections:
- wire segments 972 -> 1021
Other:
- note added: "C9 is not a GPIO on F12."
- note added: "DEAD"
- note added: "ERRATA RevA"
- note added: "FIXME: C9 is not a GPIO on F12.\nRemove pin and move LED to C8"
- moved on the sheet: U2A, U2F

Commit message: more errata
Connections:
- wire segments 1021 -> 1054
Other:
- moved on the sheet: U2F
Changed lines of the file:
@@
 	1    0    0    -1
 $EndComp
-Text GLabel 14500 16750 0    50   Input ~ 0
+Text GLabel 14500 16850 0    50   Input ~ 0
 CLK_16MHz
 Text Notes 1250 16350 0    197  ~ 0
@@
 L lfe5bg381:LFE5U-85F-6BG381C U2
 U 6 1 674D2D73
-P 15250 15950
-F 0 "U2" H 15250 16937 60  0000 C CNN
-F 1 "LFE5U-85F-6BG381C" H 15250 16831 60  0000 C CNN
-F 2 "lfe5bg381:BGA-381_pitch0.8mm_dia0.4mm" H 14200 16900 60  0001 C CNN
-F 3 "" H 14200 16900 60  0000 C CNN
-	6    15250 15950
+P 15650 16050
+F 0 "U2" H 15650 17037 60  0000 C CNN
+F 1 "LFE5U-85F-6BG381C" H 15650 16931 60  0000 C CNN
+F 2 "lfe5bg381:BGA-381_pitch0.8mm_dia0.4mm" H 14600 17000 60  0001 C CNN
+F 3 "" H 14600 17000 60  0000 C CNN
+	6    15650 16050
 	1    0    0    -1
 $EndComp
@@
 Text Label 8850 17050 2    50   ~ 0
 WIDE_39
-Text Label 16000 16750 0    50   ~ 0
+Text Label 16400 16850 0    50   ~ 0
 WIDE_1
-Text Label 16000 16650 0    50   ~ 0
+Text Label 16400 16750 0    50   ~ 0
 WIDE_3
-Text Label 14500 16350 2    50   ~ 0
+Text Label 14900 16450 2    50   ~ 0
 WIDE_5
-Text Label 14500 16150 2    50   ~ 0
+Text Label 14900 16250 2    50   ~ 0
 WIDE_7
-Text Label 16000 16050 0    50   ~ 0
+Text Label 16400 16150 0    50   ~ 0
 WIDE_9
-Text Label 14500 15450 2    50   ~ 0
+Text Label 14900 15550 2    50   ~ 0
 WIDE_11
-Text Label 14500 15650 2    50   ~ 0
+Text Label 14900 15750 2    50   ~ 0
 WIDE_13
-Text Label 14500 15350 2    50   ~ 0
+Text Label 14900 15450 2    50   ~ 0
 WIDE_15
-Text Label 14500 15550 2    50   ~ 0
+Text Label 14900 15650 2    50   ~ 0
 WIDE_17
-Text Label 16000 15350 0    50   ~ 0
+Text Label 16400 15450 0    50   ~ 0
 WIDE_19
-Text Label 16000 15250 0    50   ~ 0
+Text Label 16400 15350 0    50   ~ 0
 WIDE_21
 Text Label 11800 16450 2    50   ~ 0
@@
 Text Label 11800 15350 2    50   ~ 0
 WIDE_39
-Text Label 14500 16650 2    50   ~ 0
+Text Label 14900 16750 2    50   ~ 0
 WIDE_2
-Text Label 16000 16250 0    50   ~ 0
+Text Label 16400 16350 0    50   ~ 0
 WIDE_4
-Text Label 16000 16350 0    50   ~ 0
+Text Label 16400 16450 0    50   ~ 0
 WIDE_6
-Text Label 16000 16150 0    50   ~ 0
+Text Label 16400 16250 0    50   ~ 0
 WIDE_8
-Text Label 14500 16050 2    50   ~ 0
+Text Label 14900 16150 2    50   ~ 0
 WIDE_10
-Text Label 14500 16250 2    50   ~ 0
+Text Label 14900 16350 2    50   ~ 0
 WIDE_12
-Text Label 16000 15450 0    50   ~ 0
+Text Label 16400 15550 0    50   ~ 0
 WIDE_14
-Text Label 16000 15650 0    50   ~ 0
+Text Label 16400 15750 0    50   ~ 0
 WIDE_16
-Text Label 16000 15550 0    50   ~ 0
+Text Label 16400 15650 0    50   ~ 0
 WIDE_18
-Text Label 14500 15750 2    50   ~ 0
+Text Label 14900 15850 2    50   ~ 0
 WIDE_20
-Text Label 14500 15250 2    50   ~ 0
+Text Label 14900 15350 2    50   ~ 0
 WIDE_22
-Text Label 16000 15750 0    50   ~ 0
+Text Label 16400 15850 0    50   ~ 0
 WIDE_24
 Text Label 13300 16450 0    50   ~ 0
@@
 Text Label 5700 11750 0    50   ~ 0
 FLASH_MOSI
-NoConn ~ 14500 15850
-NoConn ~ 14500 15950
-NoConn ~ 14500 16450
-NoConn ~ 14500 16550
-NoConn ~ 16000 16450
-NoConn ~ 16000 15950
-NoConn ~ 16000 15850
+NoConn ~ 14900 15950
+NoConn ~ 14900 16050
+NoConn ~ 14900 16550
+NoConn ~ 14900 16650
+NoConn ~ 16400 16550
+NoConn ~ 16400 16050
+NoConn ~ 16400 15950
 NoConn ~ 10850 13150
 NoConn ~ 10850 13250
@@
 Wire Wire Line
 	5800 1600 5800 1650
-Text GLabel 16000 16550 2    50   Input ~ 0
+Text GLabel 16800 16650 2    50   Input ~ 0
 FT_GPIO1
 $Comp
@@
 Wire Notes Line
 	11350 16650 11200 16650
+Wire Wire Line
+	13300 15350 13700 15350
+Wire Wire Line
+	13300 15450 13700 15450
+Wire Wire Line
+	13300 15550 13700 15550
+Wire Wire Line
+	13300 15650 13700 15650
+Wire Wire Line
+	13300 15850 13700 15850
+Wire Wire Line
+	13300 15950 13700 15950
+Wire Wire Line
+	13300 16150 13700 16150
+Wire Wire Line
+	13300 16450 13700 16450
+Wire Wire Line
+	14900 15350 14500 15350
+Wire Wire Line
+	14900 15450 14500 15450
+Wire Wire Line
+	14900 15550 14500 15550
+Wire Wire Line
+	14900 15650 14500 15650
+Wire Wire Line
+	14900 15750 14500 15750
+Wire Wire Line
+	14900 15850 14500 15850
+Wire Wire Line
+	14900 16150 14500 16150
+Wire Wire Line
+	14900 16250 14500 16250
+Wire Wire Line
+	14900 16350 14500 16350
+Wire Wire Line
+	14900 16450 14500 16450
+Wire Wire Line
+	14900 16750 14500 16750
+Wire Wire Line
+	16400 15350 16800 15350
+Wire Wire Line
+	16400 15450 16800 15450
+Wire Wire Line
+	16400 15550 16800 15550
+Wire Wire Line
+	16400 15650 16800 15650
+Wire Wire Line
+	16400 15750 16800 15750
+Wire Wire Line
+	16400 15850 16800 15850
+Wire Wire Line
+	16400 16150 16800 16150
+Wire Wire Line
+	16400 16250 16800 16250
+Wire Wire Line
+	16400 16350 16800 16350
+Wire Wire Line
+	16400 16450 16800 16450
+Wire Wire Line
+	16400 16750 16800 16750
+Wire Wire Line
+	16400 16850 16800 16850
+Wire Wire Line
+	16800 16650 16400 16650
+Wire Wire Line
+	14500 16850 14900 16850
 Wire Bus Line
 	18150 9200 21550 9200
@@
 	12700 7100 12700 9100
 Wire Bus Line
-	12950 12350 12950 14200
-Wire Bus Line
-	21650 12550 21650 14200
+	10150 12350 10150 14200
 Wire Bus Line
 	18850 12750 18850 14200
 Wire Bus Line
-	10150 12350 10150 14200
+	21650 12550 21650 14200
 Wire Bus Line
-	19050 6500 19050 9100
+	12950 12350 12950 14200
 Wire Bus Line
-	14350 11350 14350 14200
+	21650 6500 21650 9100
 Wire Bus Line
 	17650 11350 17650 14200
 Wire Bus Line
-	21650 6500 21650 9100
+	14350 11350 14350 14200
+Wire Bus Line
+	19050 6500 19050 9100
 Wire Bus Line
 	18050 6500 18050 9100

Commit message: Add BODGE information
Other:
- note added: "BODGE: swap FT_RD_N with FT_CLK (R50 <-> R36)\nTODO: Route FT_CLK to a clock pin *sigh*"
- note added: "C9 is not a GPIO on F12.\nFT_CLK is not routed to a clock pin. Can be fixed with a bodge wire on RevA! (R50 <-> R36)"
- note removed: "C9 is not a GPIO on F12."
Changed lines of the file:
@@
 ERRATA RevA
 Text Notes 23900 5000 0    50   ~ 0
-C9 is not a GPIO on F12.
+C9 is not a GPIO on F12.\nFT_CLK is not routed to a clock pin. Can be fixed with a bodge wire on RevA! (R50 <-> R36)
 Text Notes 11700 17050 0    50   ~ 0
 FIXME: C9 is not a GPIO on F12.\nRemove pin and move LED to C8
@@
 Wire Bus Line
 	18050 6500 18050 9100
+Text Notes 17200 5900 0    79   ~ 0
+BODGE: swap FT_RD_N with FT_CLK (R50 <-> R36)\nTODO: Route FT_CLK to a clock pin *sigh*
 $EndSCHEMATC

Commit message: Clean up the schematic a bit
Connections:
- wire segments 1054 -> 1103
- no-connect marks 93 -> 90
Other:
- note added: "33 = NC"
- note added: "C9 is not a GPIO on ECP5 F12 and some other variants.\nFT_CLK is not routed to a clock pin. Can be fixed with a bodge wire on RevA! (R50 <-> R36)"
- note added: "PMODs"
- note added: "Wide connector"
- note removed: "C9 is not a GPIO on F12.\nFT_CLK is not routed to a clock pin. Can be fixed with a bodge wire on RevA! (R50 <-> R36)"
- note removed: "DEAD"
- moved on the sheet: D1, D10, D2, D3, D4, D5, D6, D7, D8, D9, J10, J4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

Commit message: Add errata for JTAG connector
Other:
- note added: "- C9 is not a GPIO on ECP5 F12 and some other variants.\n\n- FT_CLK is not routed to a clock pin. Can be fixed with a bodge wire on RevA! (R50 <-> R36)\n\n- JTAG connector has a funky footprint on the PCB because CCW vs Odd/Even pinout on the symbol vs footprint.\n PCB silk screen is accurate so don't worry - it's just a stupid pinout."
- note added: "FIXME: Use ODD-EVEN in RevB."
- note removed: "C9 is not a GPIO on ECP5 F12 and some other variants.\nFT_CLK is not routed to a clock pin. Can be fixed with a bodge wire on RevA! (R50 <-> R36)"
Changed lines of the file:
@@
 Text Notes 23750 4700 0    394  ~ 79
 ERRATA RevA
-Text Notes 23900 5000 0    50   ~ 0
-C9 is not a GPIO on ECP5 F12 and some other variants.\nFT_CLK is not routed to a clock pin. Can be fixed with a bodge wire on RevA! (R50 <-> R36)
+Text Notes 23900 5300 0    50   ~ 0
+- C9 is not a GPIO on ECP5 F12 and some other variants.\n\n- FT_CLK is not routed to a clock pin. Can be fixed with a bodge wire on RevA! (R50 <-> R36)\n\n- JTAG connector has a funky footprint on the PCB because CCW vs Odd/Even pinout on the symbol vs footprint.\n   PCB silk screen is accurate so don't worry - it's just a stupid pinout.
 Text Notes 15550 17050 0    50   ~ 0
 FIXME: C9 is not a GPIO on F12.\nRemove pin and move LED to C8
@@
 Wire Bus Line
 	7050 16650 7050 21400
+Text Notes 2050 11700 0    50   ~ 0
+FIXME: Use ODD-EVEN in RevB.
 $EndSCHEMATC

Commit message: Woop! Can send I2C data
Parts:
- added U4: LFE5UM-45F-6BG381C, lfe5bg381:BGA-381_pitch0.8mm_dia0.4mm, symbol lfe5bg381:LFE5UM-45F-6BG381C
- J2: symbol Connector:USB_C_Receptacle -> Kilsyth-rescue:USB_C_Receptacle-Connector
- Y1: symbol Device:Crystal_GND24_Small -> Kilsyth-rescue:Crystal_GND24_Small-Device
Changed lines of the file:
@@
 EESchema Schematic File Version 4
 LIBS:Kilsyth-cache
-EELAYER 26 0
+EELAYER 29 0
 EELAYER END
 $Descr A1 33110 23386
@@
 $EndComp
 $Comp
-L Connector:USB_C_Receptacle J2
+L Kilsyth-rescue:USB_C_Receptacle-Connector J2
 U 1 1 5FDA1710
 P 9300 7400
@@
 $EndComp
 $Comp
-L Device:Crystal_GND24_Small Y1
+L Kilsyth-rescue:Crystal_GND24_Small-Device Y1
 U 1 1 64D1A925
 P 14200 7950
@@
 Text Notes 13300 14950 0    197  ~ 0
 Wide connector
+Text Notes 2050 11700 0    50   ~ 0
+FIXME: Use ODD-EVEN in RevB.
 Wire Bus Line
 	18150 9200 21550 9200
@@
 Wire Bus Line
 	7050 16650 7050 21400
-Text Notes 2050 11700 0    50   ~ 0
-FIXME: Use ODD-EVEN in RevB.
+$Comp
+L lfe5bg381:LFE5UM-45F-6BG381C U4
+U 8 1 5CEB4B25
+P 15650 20500
+F 0 "U4" H 15650 21793 60  0000 C CNN
+F 1 "LFE5UM-45F-6BG381C" H 15650 21687 60  0000 C CNN
+F 2 "lfe5bg381:BGA-381_pitch0.8mm_dia0.4mm" H 15650 21581 60  0000 C CNN
+F 3 "" H 14600 21450 60  0000 C CNN
+	8    15650 20500
+	1    0    0    -1
+$EndComp
 $EndSCHEMATC
