File: hardware/RevB/Kilsyth.kicad_pcb (KiCad board)
At the start: 4 copper layers, 95 x 80 mm, 152 parts, among them J1 Conn_JTAG, J10 PUSB3FR4Z, J11 PUSB3FR4Z, J12 PUSB3FR4Z, J2 DX07S024JJ2, J3 PUSB3FR4Z, J4 PUSB3FR4Z, J5 PUSB3FR4Z, J6 DX07S024JJ2, J7 DX07S024JJ2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

Commit message: Add usb-c-breakout
Parts:
- added J13: PUSB3FR4Z, PUSB3FR4Z:PUSB3FR4Z, F.Cu at (180.9, 89.0)
- added J14: PUSB3FR4Z, PUSB3FR4Z:PUSB3FR4Z, F.Cu at (170.0, 104.0)
- added TP5: TestPoint, TestPoint:TestPoint_Pad_D1.0mm, F.Cu at (180.2, 91.8)
- added U6: PI5USB30213A, kilsyth_extra:PI5USB30213A, F.Cu at (170.0, 99.3)
- moved Y1 116.9 mm to (184.6, 89.1), turned to 0 degrees
- moved J7 68.3 mm to (173.2, 91.0)
- moved J6 66.3 mm to (162.3, 100.2)
Connections:
- C28 pad 2: (no net) -> Net-(C28-Pad2)
- C30 pad 2: (no net) -> Net-(C30-Pad2)
- C31 pad 2: (no net) -> Net-(C31-Pad2)
- C7 pad 2: (no net) -> Net-(C7-Pad2)
- FB1 pad 1: +5V -> VBUS
- FB1 pad 2: +5V -> Net-(FB1-Pad2)
- J2 pad A4: +5V -> Net-(FB1-Pad2)
- J2 pad A5: (no net) -> /CC1
- J2 pad A9: +5V -> Net-(FB1-Pad2)
- J2 pad B4: +5V -> Net-(FB1-Pad2)
- J2 pad B5: (no net) -> /CC2
- J2 pad B9: +5V -> Net-(FB1-Pad2)
- J4 pad 4: Net-(J4-Pad4) -> /CC2
- J4 pad 5: Net-(J4-Pad5) -> /CC1
- J4 pad 6: Net-(J4-Pad5) -> /CC1
- J4 pad 7: Net-(J4-Pad4) -> /CC2
- J6 pad A5: (no net) -> /USBC0_CC1
- J6 pad B5: (no net) -> /USBC0_CC2
- J7 pad A5: (no net) -> /USBC1_CC1
- J7 pad B5: (no net) -> /USBC1_CC2
- R16 pad 1: +5V -> VBUS
- R16 pad 2: (no net) -> Net-(R16-Pad2)
- R21 pad 1: (no net) -> +1V8
- R27 pad 2: +5V -> VBUS
Routing:
- net (no net): track 1803.7 -> 1772.2 mm, vias 78 -> 73
- net /CC1: track 0.00 -> 13.5 mm, vias 0 -> 2
- net Net-(C31-Pad2): track 0.00 -> 9.79 mm, vias 0 -> 2
- net +5V: track 20.0 -> 11.0 mm, vias 21 -> 18
- net Net-(FB1-Pad2): track 0.00 -> 8.97 mm, vias 0 -> 3
- net Net-(C30-Pad2): track 0.00 -> 8.19 mm, vias 0 -> 1
