File: hardware/RevB/Kilsyth.sch (KiCad schematic (older format))
At the start: 155 parts, among them J1 Conn_JTAG, J10 PUSB3FR4Z, J11 PUSB3FR4Z, J12 PUSB3FR4Z, J13 PUSB3FR4Z, J14 PUSB3FR4Z, J2 DX07S024JJ2, J3 PUSB3FR4Z, J4 PUSB3FR4Z, J5 PUSB3FR4Z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

Commit message: Add usb-c-breakout
Parts:
- U6: footprint (none) -> kilsyth_extra:PI5USB30213A
Changed lines of the file:
@@
 Text Label 15550 21000 0    50   ~ 0
 REFCLK_D0_P
-$Comp
-L PI5USB30213A:PI5USB30213A U6
-U 1 1 5D0FB9EA
-P 11800 5450
-F 0 "U6" H 11350 4400 50  0000 C CNN
-F 1 "PI5USB30213A" H 12200 4350 50  0000 C CNN
-F 2 "" H 11800 5450 50  0001 C CNN
-F 3 "" H 11800 5450 50  0001 C CNN
-	1    11800 5450
-	1    0    0    -1
-$EndComp
 NoConn ~ 11100 5050
 $Comp
@@
 	0    1    1    0
 $EndComp
-Wire Bus Line
-	19450 9350 22850 9350
-Wire Bus Line
-	12950 5750 12950 7450
-Wire Bus Line
-	15750 6850 15750 7450
-Wire Bus Line
-	20350 4850 20350 9250
-Wire Bus Line
-	22950 4850 22950 9250
-Wire Bus Line
-	19350 4850 19350 9250
 Text Notes 28750 1050 0    394  ~ 79
 Kilsyth RevB
+Wire Bus Line
+	19450 9350 22850 9350
+Wire Bus Line
+	12950 5750 12950 7450
+Wire Bus Line
+	15750 6850 15750 7450
+Wire Bus Line
+	20350 4850 20350 9250
+Wire Bus Line
+	22950 4850 22950 9250
+Wire Bus Line
+	19350 4850 19350 9250
+$Comp
+L PI5USB30213A:PI5USB30213A U6
+U 1 1 5DBFCED5
+P 11800 5450
+F 0 "U6" H 12250 4400 50  0000 C CNN
+F 1 "PI5USB30213A" H 12300 6400 50  0000 C CNN
+F 2 "kilsyth_extra:PI5USB30213A" H 11800 5450 50  0001 C CNN
+F 3 "" H 11800 5450 50  0001 C CNN
+	1    11800 5450
+	1    0    0    -1
+$EndComp
 $EndSCHEMATC

Commit message: Add note about USB2422
Other:
- note added: "- FT_CLK must be routed to a clock input.\n\n- Route HDMI traces properly...\n\n- Need extra oscillator?\n\n- Use USB2422 + SAMD11 or similar for jtag!\n Connect the FT's HS pins and SAMD11 on the hub."
- note removed: "- FT_CLK must be routed to a clock input.\n\n- Route HDMI traces properly...\n\n- Need extra oscillator?"
Changed lines of the file:
@@
 EESchema Schematic File Version 4
-LIBS:Kilsyth-cache
 EELAYER 30 0
 EELAYER END
@@
 Notes to self
 Text Notes 23900 5350 0    50   ~ 0
-- FT_CLK must be routed to a clock input.\n\n- Route HDMI traces properly...\n\n- Need extra oscillator?
+- FT_CLK must be routed to a clock input.\n\n- Route HDMI traces properly...\n\n- Need extra oscillator?\n\n- Use USB2422 + SAMD11 or similar for jtag!\n    Connect the FT's HS pins and SAMD11 on the hub.
 Wire Notes Line
 	7750 14550 23200 14550
@@
 Text Notes 28750 1050 0    394  ~ 79
 Kilsyth RevB
+$Comp
+L PI5USB30213A:PI5USB30213A U6
+U 1 1 5DBFCED5
+P 11800 5450
+F 0 "U6" H 12250 4400 50  0000 C CNN
+F 1 "PI5USB30213A" H 12300 6400 50  0000 C CNN
+F 2 "kilsyth_extra:PI5USB30213A" H 11800 5450 50  0001 C CNN
+F 3 "" H 11800 5450 50  0001 C CNN
+	1    11800 5450
+	1    0    0    -1
+$EndComp
 Wire Bus Line
 	19450 9350 22850 9350
@@
 Wire Bus Line
 	19350 4850 19350 9250
-$Comp
-L PI5USB30213A:PI5USB30213A U6
-U 1 1 5DBFCED5
-P 11800 5450
-F 0 "U6" H 12250 4400 50  0000 C CNN
-F 1 "PI5USB30213A" H 12300 6400 50  0000 C CNN
-F 2 "kilsyth_extra:PI5USB30213A" H 11800 5450 50  0001 C CNN
-F 3 "" H 11800 5450 50  0001 C CNN
-	1    11800 5450
-	1    0    0    -1
-$EndComp
 $EndSCHEMATC
